File: ControlBoard.sch (EAGLE design)
At the start: 0 parts

Commit message: futher effort and set 3v3 analog
Parts:
- added C1: 1u, rcl:C-EUC0805
- added C2, C3: (no value), rcl:C-EUC0805
- added IC1: TL074P, linear:TL074P
- added IC2: LM4041B12DBZ, texas:LM4041B12DBZ
- added R1: EVUF2A, pot:EVUF2A
- added R2: 100k, rcl:R-EU_R0805
- added R3: 33k, rcl:R-EU_R0805
- added R4: 200k, rcl:R-EU_R0805
- added R5, R6, R7, R8, R9: 10k, rcl:R-EU_R0805
- added SV1, SV2, SV3, SV4: (no value), con-lstb:MA08-2
- added U$1, U$10, U$11, U$12, U$13, U$2, U$3, U$4, U$5, U$6, U$7, U$8, U$9: WQP-PJ301M-12_JACK, thonkiconn:WQP-PJ301M-12_JACK
- added U1, U2: PEC11R-4315F-N0012, SamacSys_Parts:PEC11R-4315F-N0012
Connections:
- new net +3V3: R5.1, R8.1, R9.1
- new net -10V: R1.A
- new net 1V2REF: IC1A.+IN
- new net AGND: SV1.1, SV1.10, SV1.13, SV1.14, SV1.2, SV1.5, SV1.6, SV1.9, SV2.1, SV2.10, SV2.13, SV2.14, SV2.2, SV2.5, SV2.6, SV2.9, SV4.1, SV4.10, SV4.13, SV4.14, SV4.2, SV4.5, SV4.6, SV4.9
- new net CV0: C1.2, IC1A.OUT, R3.2
- new net ENCODER00: C2.1, R6.1
- new net ENCODER01: C3.1, R7.2
- new net ENCODER0SW: R5.2, U1.COM
- new net GND: C2.2, C3.2, R1.E, U$1.1, U$1.3, U1.B, U1.NO
- new net IN0+: SV1.15
- new net IN0-: SV1.16
- new net IN1+: SV1.11
- new net IN1-: SV1.12
- new net IN2+: SV1.7
- new net IN2-: SV1.8
- new net IN3+: SV1.3
- new net IN3-: SV1.4
- new net N$1: R2.1, U$1.2
- new net N$2: R1.S, R4.1
- new net N$3: C1.1, IC1A.-IN, R2.2, R3.1, R4.2
- new net N$4: R6.2, R8.2, U1.A
- new net N$5: R7.1, R9.2, U1.C
- new net OUT0+: SV2.15
- new net OUT0-: SV2.16
- new net OUT1+: SV2.11
- new net OUT1-: SV2.12
- new net OUT2+: SV2.7
- new net OUT2-: SV2.8
- new net OUT3+: SV2.3
- new net OUT3-: SV2.4
- new net OUT4+: SV4.15
- new net OUT4-: SV4.16
- new net OUT5+: SV4.11
- new net OUT5-: SV4.12
- new net OUT6+: SV4.7
- new net OUT6-: SV4.8
- new net OUT7+: SV4.3
- new net OUT7-: SV4.4
Other:
- note added: "Audio From DSP Board"
- note added: "Audio To DSP Board"
- note added: "LEDS"
