File: DSPBoard.sch (EAGLE design)
At the start: 450 parts, among them IC1 AD1939WBSTZ, IC10 LM833D, IC11 LM833D, IC12 TL074D, IC13 CD74HC4094M96, IC14 CD74HC4094M96, IC17 CD74HC4094M96, IC18 CD74HC4094M96, IC2 25AA1024-I_SM, IC3 LM4040B10DBZ, IC4 LM833D, IC5 LM833D, IC6 LM833D, IC7 LM833D, IC8 LM833D, IC9 LM833D, U1 LM11173.3NOPB, U2 PEC11R-4315F-N0012, U3 PEC11R-4315F-N0012, X1 2510-, Y1 12.288MHz

Commit message: Ready to lay out
Parts:
- added D2, D3, D4, D5, D6, D7, D8: BAV99,215, SamacSys_Parts:BAV99,215
Connections:
- new net N$235: D1.ANODE_(DIODE_1), D2.ANODE_(DIODE_1)
- new net N$236: D1.CATHODE_(DIODE_2), D2.CATHODE_(DIODE_2)
- new net N$237: D3.ANODE_(DIODE_1), D4.ANODE_(DIODE_1)
- new net N$238: D3.CATHODE_(DIODE_2), D4.CATHODE_(DIODE_2)
- new net N$239: D5.ANODE_(DIODE_1), D6.ANODE_(DIODE_1)
- new net N$240: D5.CATHODE_(DIODE_2), D6.CATHODE_(DIODE_2)
- new net N$241: D7.ANODE_(DIODE_1), D8.ANODE_(DIODE_1)
- new net N$242: D7.CATHODE_(DIODE_2), D8.CATHODE_(DIODE_2)
- net AIN0+: now also D2.CATHODE_(DIODE_1),_ANODE_(DIODE_2)
- net AIN0-: now also D1.CATHODE_(DIODE_1),_ANODE_(DIODE_2)
- net AIN1+: now also D4.CATHODE_(DIODE_1),_ANODE_(DIODE_2)
- net AIN1-: now also D3.CATHODE_(DIODE_1),_ANODE_(DIODE_2)
- net AIN2+: now also D6.CATHODE_(DIODE_1),_ANODE_(DIODE_2)
- net AIN2-: now also D5.CATHODE_(DIODE_1),_ANODE_(DIODE_2)
- net AIN3+: now also D8.CATHODE_(DIODE_1),_ANODE_(DIODE_2)
- net AIN3-: now also D7.CATHODE_(DIODE_1),_ANODE_(DIODE_2)
Other:
- moved on the sheet: D1
Changed lines of the file:
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@@
 <part name="+3V20" library="supply1" library_urn="urn:adsk.eagle:library:371" deviceset="+3V3" device=""/>
 <part name="D1" library="SamacSys_Parts" deviceset="BAV99,215" device=""/>
+<part name="D2" library="SamacSys_Parts" deviceset="BAV99,215" device=""/>
+<part name="D3" library="SamacSys_Parts" deviceset="BAV99,215" device=""/>
+<part name="D4" library="SamacSys_Parts" deviceset="BAV99,215" device=""/>
+<part name="D5" library="SamacSys_Parts" deviceset="BAV99,215" device=""/>
+<part name="D6" library="SamacSys_Parts" deviceset="BAV99,215" device=""/>
+<part name="D7" library="SamacSys_Parts" deviceset="BAV99,215" device=""/>
+<part name="D8" library="SamacSys_Parts" deviceset="BAV99,215" device=""/>
 </parts>
 <sheets>
@@
 <attribute name="VALUE" x="182.88" y="45.72" size="1.778" layer="96"/>
 </instance>
-<instance part="D1" gate="G$1" x="213.36" y="121.92" smashed="yes">
-<attribute name="NAME" x="293.37" y="129.54" size="1.778" layer="95" align="center-left"/>
-<attribute name="VALUE" x="293.37" y="127" size="1.778" layer="96" align="center-left"/>
+<instance part="D1" gate="G$1" x="294.64" y="154.94" smashed="yes">
+<attribute name="NAME" x="374.65" y="162.56" size="1.778" layer="95" align="center-left"/>
+<attribute name="VALUE" x="374.65" y="160.02" size="1.778" layer="96" align="center-left"/>
+</instance>
+<instance part="D2" gate="G$1" x="294.64" y="142.24" smashed="yes">
+<attribute name="NAME" x="374.65" y="149.86" size="1.778" layer="95" align="center-left"/>
+<attribute name="VALUE" x="374.65" y="147.32" size="1.778" layer="96" align="center-left"/>
+</instance>
+<instance part="D3" gate="G$1" x="294.64" y="129.54" smashed="yes">
+<attribute name="NAME" x="374.65" y="137.16" size="1.778" layer="95" align="center-left"/>
+<attribute name="VALUE" x="374.65" y="134.62" size="1.778" layer="96" align="center-left"/>
+</instance>
+<instance part="D4" gate="G$1" x="294.64" y="116.84" smashed="yes">
+<attribute name="NAME" x="374.65" y="124.46" size="1.778" layer="95" align="center-left"/>
+<attribute name="VALUE" x="374.65" y="121.92" size="1.778" layer="96" align="center-left"/>
+</instance>
+<instance part="D5" gate="G$1" x="294.64" y="104.14" smashed="yes">
+<attribute name="NAME" x="374.65" y="111.76" size="1.778" layer="95" align="center-left"/>
+<attribute name="VALUE" x="374.65" y="109.22" size="1.778" layer="96" align="center-left"/>
+</instance>
+<instance part="D6" gate="G$1" x="294.64" y="91.44" smashed="yes">
+<attribute name="NAME" x="374.65" y="99.06" size="1.778" layer="95" align="center-left"/>
+<attribute name="VALUE" x="374.65" y="96.52" size="1.778" layer="96" align="center-left"/>
+</instance>
+<instance part="D7" gate="G$1" x="294.64" y="78.74" smashed="yes">
+<attribute name="NAME" x="374.65" y="86.36" size="1.778" layer="95" align="center-left"/>
+<attribute name="VALUE" x="374.65" y="83.82" size="1.778" layer="96" align="center-left"/>
+</instance>
+<instance part="D8" gate="G$1" x="294.64" y="66.04" smashed="yes">
+<attribute name="NAME" x="374.65" y="73.66" size="1.778" layer="95" align="center-left"/>
+<attribute name="VALUE" x="374.65" y="71.12" size="1.778" layer="96" align="center-left"/>
 </instance>
 </instances>
@@
 <junction x="121.92" y="165.1"/>
 </segment>
+<segment>
+<pinref part="D1" gate="G$1" pin="CATHODE_(DIODE_1),_ANODE_(DIODE_2)"/>
+<wire x1="378.46" y1="154.94" x2="388.62" y2="154.94" width="0.1524" layer="91"/>
+<label x="388.62" y="154.94" size="2.54" layer="95" xref="yes"/>
+</segment>
 </net>
 <net name="AIN0+" class="0">
@@
 <junction x="121.92" y="134.62"/>
 </segment>
+<segment>
+<pinref part="D2" gate="G$1" pin="CATHODE_(DIODE_1),_ANODE_(DIODE_2)"/>
+<wire x1="378.46" y1="142.24" x2="388.62" y2="142.24" width="0.1524" layer="91"/>
+<label x="388.62" y="142.24" size="2.54" layer="95" xref="yes"/>
+</segment>
 </net>
 <net name="N$9" class="0">
@@
 <junction x="121.92" y="96.52"/>
 </segment>
+<segment>
+<pinref part="D3" gate="G$1" pin="CATHODE_(DIODE_1),_ANODE_(DIODE_2)"/>
+<wire x1="378.46" y1="129.54" x2="388.62" y2="129.54" width="0.1524" layer="91"/>
+<label x="388.62" y="129.54" size="2.54" layer="95" xref="yes"/>
+</segment>
 </net>
 <net name="AIN1+" class="0">
@@
 <junction x="121.92" y="66.04"/>
 </segment>
+<segment>
+<pinref part="D4" gate="G$1" pin="CATHODE_(DIODE_1),_ANODE_(DIODE_2)"/>
+<wire x1="378.46" y1="116.84" x2="388.62" y2="116.84" width="0.1524" layer="91"/>
+<label x="388.62" y="116.84" size="2.54" layer="95" xref="yes"/>
+</segment>
 </net>
 <net name="AIN2-" class="0">
@@
 <junction x="261.62" y="167.64"/>
 </segment>
+<segment>
+<pinref part="D5" gate="G$1" pin="CATHODE_(DIODE_1),_ANODE_(DIODE_2)"/>
+<wire x1="378.46" y1="104.14" x2="388.62" y2="104.14" width="0.1524" layer="91"/>
+<label x="388.62" y="104.14" size="2.54" layer="95" xref="yes"/>
+</segment>
 </net>
 <net name="AIN2+" class="0">
@@
 <junction x="261.62" y="137.16"/>
 </segment>
+<segment>
+<pinref part="D6" gate="G$1" pin="CATHODE_(DIODE_1),_ANODE_(DIODE_2)"/>
+<wire x1="378.46" y1="91.44" x2="388.62" y2="91.44" width="0.1524" layer="91"/>
+<label x="388.62" y="91.44" size="2.54" layer="95" xref="yes"/>
+</segment>
 </net>
 <net name="AIN3-" class="0">
@@
 <junction x="261.62" y="96.52"/>
 </segment>
+<segment>
+<pinref part="D7" gate="G$1" pin="CATHODE_(DIODE_1),_ANODE_(DIODE_2)"/>
+<wire x1="378.46" y1="78.74" x2="388.62" y2="78.74" width="0.1524" layer="91"/>
+<label x="388.62" y="78.74" size="2.54" layer="95" xref="yes"/>
+</segment>
 </net>
 <net name="AIN3+" class="0">
@@
 <junction x="261.62" y="66.04"/>
 </segment>
+<segment>
+<pinref part="D8" gate="G$1" pin="CATHODE_(DIODE_1),_ANODE_(DIODE_2)"/>
+<wire x1="378.46" y1="66.04" x2="388.62" y2="66.04" width="0.1524" layer="91"/>
+<label x="388.62" y="66.04" size="2.54" layer="95" xref="yes"/>
+</segment>
+</net>
+<net name="N$235" class="0">
+<segment>
+<pinref part="D1" gate="G$1" pin="ANODE_(DIODE_1)"/>
+<wire x1="294.64" y1="154.94" x2="289.56" y2="154.94" width="0.1524" layer="91"/>
+<wire x1="289.56" y1="154.94" x2="289.56" y2="142.24" width="0.1524" layer="91"/>
+<pinref part="D2" gate="G$1" pin="ANODE_(DIODE_1)"/>
+<wire x1="289.56" y1="142.24" x2="294.64" y2="142.24" width="0.1524" layer="91"/>
+</segment>
+</net>
+<net name="N$236" class="0">
+<segment>
+<pinref part="D1" gate="G$1" pin="CATHODE_(DIODE_2)"/>
+<wire x1="294.64" y1="152.4" x2="292.1" y2="152.4" width="0.1524" layer="91"/>
+<wire x1="292.1" y1="152.4" x2="292.1" y2="139.7" width="0.1524" layer="91"/>
+<pinref part="D2" gate="G$1" pin="CATHODE_(DIODE_2)"/>
+<wire x1="292.1" y1="139.7" x2="294.64" y2="139.7" width="0.1524" layer="91"/>
+</segment>
+</net>
+<net name="N$237" class="0">
+<segment>
+<pinref part="D3" gate="G$1" pin="ANODE_(DIODE_1)"/>
+<wire x1="294.64" y1="129.54" x2="289.56" y2="129.54" width="0.1524" layer="91"/>
+<wire x1="289.56" y1="129.54" x2="289.56" y2="116.84" width="0.1524" layer="91"/>
+<pinref part="D4" gate="G$1" pin="ANODE_(DIODE_1)"/>
+<wire x1="289.56" y1="116.84" x2="294.64" y2="116.84" width="0.1524" layer="91"/>
+</segment>
+</net>
+<net name="N$238" class="0">
+<segment>
+<pinref part="D3" gate="G$1" pin="CATHODE_(DIODE_2)"/>
+<wire x1="294.64" y1="127" x2="292.1" y2="127" width="0.1524" layer="91"/>
+<wire x1="292.1" y1="127" x2="292.1" y2="114.3" width="0.1524" layer="91"/>
+<pinref part="D4" gate="G$1" pin="CATHODE_(DIODE_2)"/>
+<wire x1="292.1" y1="114.3" x2="294.64" y2="114.3" width="0.1524" layer="91"/>
+</segment>
+</net>
+<net name="N$239" class="0">
+<segment>
+<pinref part="D5" gate="G$1" pin="ANODE_(DIODE_1)"/>
+<wire x1="294.64" y1="104.14" x2="289.56" y2="104.14" width="0.1524" layer="91"/>
+<wire x1="289.56" y1="104.14" x2="289.56" y2="91.44" width="0.1524" layer="91"/>
+<pinref part="D6" gate="G$1" pin="ANODE_(DIODE_1)"/>
+<wire x1="289.56" y1="91.44" x2="294.64" y2="91.44" width="0.1524" layer="91"/>
+</segment>
+</net>
+<net name="N$240" class="0">
+<segment>
+<pinref part="D5" gate="G$1" pin="CATHODE_(DIODE_2)"/>
+<wire x1="294.64" y1="101.6" x2="292.1" y2="101.6" width="0.1524" layer="91"/>
+<wire x1="292.1" y1="101.6" x2="292.1" y2="88.9" width="0.1524" layer="91"/>
+<pinref part="D6" gate="G$1" pin="CATHODE_(DIODE_2)"/>
+<wire x1="292.1" y1="88.9" x2="294.64" y2="88.9" width="0.1524" layer="91"/>
+</segment>
+</net>
+<net name="N$241" class="0">
+<segment>
+<pinref part="D7" gate="G$1" pin="ANODE_(DIODE_1)"/>
+<wire x1="294.64" y1="78.74" x2="289.56" y2="78.74" width="0.1524" layer="91"/>
+<wire x1="289.56" y1="78.74" x2="289.56" y2="66.04" width="0.1524" layer="91"/>
+<pinref part="D8" gate="G$1" pin="ANODE_(DIODE_1)"/>
+<wire x1="289.56" y1="66.04" x2="294.64" y2="66.04" width="0.1524" layer="91"/>
+</segment>
+</net>
+<net name="N$242" class="0">
+<segment>
+<pinref part="D7" gate="G$1" pin="CATHODE_(DIODE_2)"/>
+<wire x1="294.64" y1="76.2" x2="292.1" y2="76.2" width="0.1524" layer="91"/>
+<wire x1="292.1" y1="76.2" x2="292.1" y2="63.5" width="0.1524" layer="91"/>
+<pinref part="D8" gate="G$1" pin="CATHODE_(DIODE_2)"/>
+<wire x1="292.1" y1="63.5" x2="294.64" y2="63.5" width="0.1524" layer="91"/>
+</segment>
 </net>

Commit message: rethinking the strategy
Parts:
- added C146, C147, C150, C151: 0.1u, rcl:C-EUC0805
- added C148, C149: 100nF, rcl:C-EUC0805
- added IC15, IC16, IC19, IC20, IC21, IC22, IC23, IC24, IC25, IC26, IC27, IC28, LED_STROBE2, LED_STROBE3, LED_STROBE4, LED_STROBE5, LED_STROBE6, LED_STROBE7: CD74HC4094M96, CD74HC4094M96:CD74HC4094M96
- added IC29: TL074D, linear:TL074D
- added LED100, LED101, LED102, LED103, LED104, LED105, LED106, LED107, LED108, LED109, LED110, LED111, LED112, LED113, LED114, LED115, LED116, LED117, LED118, LED119, LED120, LED121, LED122, LED123, LED124, LED125, LED126, LED127, LED128, LED129, LED130, LED131, LED132, LED133, LED134, LED135, LED136, LED137, LED138, LED139, LED140, LED141, LED142, LED143, LED144, LED145, LED146, LED147, LED148, LED149, LED150, LED151, LED152, LED153, LED154, LED155, LED156, LED157, LED158, LED159, LED160, LED161, LED162, LED163, LED164, LED165, LED166, LED167, LED168, LED169, LED170, LED171, LED172, LED173, LED174, LED175, LED176, LED177, LED178, LED179, LED180, LED181, LED182, LED183, LED184, LED185, LED186, LED187, LED188, LED189, LED190, LED191, LED192, LED49, LED50, LED51, LED52, LED53, LED54, LED55, LED56, LED57, LED58, LED59, LED60, LED61, LED62, LED63, LED64, LED65, LED66, LED67, LED68, LED69, LED70, LED71, LED72, LED73, LED74, LED75, LED76, LED77, LED78, LED79, LED80, LED81, LED82, LED83, LED84, LED85, LED86, LED87, LED88, LED89, LED90, LED91, LED92, LED93, LED94, LED95, LED96, LED97, LED98, LED99: (no value), led:LEDCHIPLED_0805
- added R203, R204, R205, R206, R207, R208, R209, R210, R211, R212, R213, R214, R219, R220, R221, R222, R223, R224, R225, R226, R227, R228, R229, R230, R231, R232, R233, R234, R235, R236, R237, R238, R243, R244, R245, R246, R247, R248, R249, R250, R251, R252, R253, R254, R255, R256, R257, R258, R259, R260, R261, R262, R267, R268, R269, R270, R271, R272, R273, R274, R275, R276, R277, R278, R279, R280, R281, R282, R283, R284, R285, R286, R291, R292, R293, R294, R295, R296, R297, R298, R299, R300, R301, R302, R303, R304, R305, R306, R307, R308, R309, R310, R315, R316, R317, R318, R319, R320, R321, R322, R323, R324, R325, R326, R327, R328, R329, R330, R331, R332, R333, R334, R339, R340, R341, R342, R343, R344, R345, R346: 470R, rcl:R-EU_R0805
- added R215, R216, R217, R218, R239, R240, R241, R242, R263, R264, R265, R266, R287, R288, R289, R290, R311, R312, R313, R314, R335, R336, R337, R338: 470, rcl:R-EU_R0805
- added R347, R349, R350, R352, R355, R357, R359, R361: 100k, rcl:R-EU_R0805
- added R348, R351, R356, R360: 15k, rcl:R-EU_R0805
- added R353, R354, R358, R362: 200k, rcl:R-EU_R0805
- added U$22: ULN2803A, audioic:ULN2803A
- added U$24: PHOTON_SMD, Particle-Devices:PHOTON_SMD
- added U$25, U$26, U$27, U$28: WQP-PJ301M-12_JACK, thonkiconn:WQP-PJ301M-12_JACK
- added U4: SN74HC595D, SparkFun-IC-Logic:74HC595D
- added VR5, VR7: 100k, SparkFun-Resistors:POTENTIOMETER-PTH-9MM-1/20W-20%-KIT
- added VR6, VR8: 10k, SparkFun-Resistors:POTENTIOMETER-PTH-9MM-1/20W-20%-KIT
Connections:
- removed net LED_S3: IC17.DATA, IC18.QS1
- removed net LED_S4: IC17.QS1, LED_STROBE1.DATA
- new net CV4: C146.2, IC29A.OUT, R348.1
- new net CV5: C150.2, IC29B.OUT, R356.1
- new net CV6: C151.2, IC29D.OUT, R360.1
- new net CV7: C147.2, IC29C.OUT, R351.1
- new net LED_ROW_1: LED1.C, LED100.C, LED109.C, LED110.C, LED111.C, LED112.C, LED113.C, LED114.C, LED115.C, LED116.C, LED121.C, LED122.C, LED123.C, LED124.C, LED13.C, LED133.C, LED134.C, LED135.C, LED136.C, LED137.C, LED138.C, LED139.C, LED14.C, LED140.C, LED145.C, LED146.C, LED147.C, LED148.C, LED15.C, LED157.C, LED158.C, LED159.C, LED16.C, LED160.C, LED161.C, LED162.C, LED163.C, LED164.C, LED169.C, LED17.C, LED170.C, LED171.C, LED172.C, LED18.C, LED181.C, LED182.C, LED183.C, LED184.C, LED185.C, LED186.C, LED187.C, LED188.C, LED19.C, LED2.C, LED20.C, LED25.C, LED26.C, LED27.C, LED28.C, LED3.C, LED37.C, LED38.C, LED39.C, LED4.C, LED40.C, LED41.C, LED42.C, LED43.C, LED44.C, LED49.C, LED50.C, LED51.C, LED52.C, LED61.C, LED62.C, LED63.C, LED64.C, LED65.C, LED66.C, LED67.C, LED68.C, LED73.C, LED74.C, LED75.C, LED76.C, LED85.C, LED86.C, LED87.C, LED88.C, LED89.C, LED90.C, LED91.C, LED92.C, LED97.C, LED98.C, LED99.C, U$22.OUT1
- new net LED_ROW_2: U$22.OUT2
- new net LED_ROW_3: U$22.OUT3
- new net LED_ROW_4: U$22.OUT4
- new net LED_ROW_5: U$22.OUT5
- new net LED_ROW_6: U$22.OUT6
- new net LED_ROW_7: U$22.OUT7
- new net LED_ROW_8: U$22.OUT8
- new net N$234: D1.3, D3.3, D5.3, D7.3
- new net N$243: IC18.Q4, R218.1
- new net N$244: LED_STROBE2.Q4, R219.1
- new net N$245: LED_STROBE2.Q5, R220.1
- new net N$246: LED_STROBE2.Q6, R221.1
- new net N$247: LED_STROBE2.Q7, R222.1
- new net N$248: LED_STROBE2.Q3, R223.2
- new net N$249: LED_STROBE2.Q2, R224.2
- new net N$250: LED_STROBE2.Q1, R225.2
- new net N$251: LED_STROBE2.Q0, R226.2
- new net N$252: LED49.A, R203.2
- new net N$253: LED50.A, R204.2
- new net N$254: LED51.A, R205.2
- new net N$255: LED52.A, R206.2
- new net N$256: LED53.A, R207.1
- new net N$257: LED54.A, R208.1
- new net N$258: LED55.A, R209.1
- new net N$259: LED56.A, R210.1
- new net N$260: LED57.A, R211.1
- new net N$261: LED58.A, R212.1
- new net N$262: LED59.A, R213.1
- new net N$263: LED60.A, R214.1
- new net N$264: LED61.A, R215.2
- new net N$265: LED62.A, R216.2
- new net N$266: LED63.A, R217.2
- new net N$267: LED64.A, R218.2
- new net N$268: LED65.A, R219.2
- new net N$269: LED66.A, R220.2
- new net N$270: LED67.A, R221.2
- new net N$271: LED68.A, R222.2
- new net N$272: LED69.A, R223.1
- new net N$273: LED70.A, R224.1
- new net N$274: LED71.A, R225.1
- new net N$275: LED72.A, R226.1
- new net N$276: IC18.Q5, R217.1
- new net N$277: IC18.Q1, R212.2
- new net N$278: IC18.Q2, R213.2
- new net N$279: IC18.Q3, R214.2
- new net N$280: IC17.Q4, R203.1
- new net N$281: IC17.Q6, R205.1
- new net N$282: IC17.Q7, R206.1
- new net N$283: IC17.Q1, R209.2
- new net N$284: IC19.Q5, R228.1
- new net N$285: IC19.Q3, R231.2
- new net N$286: IC19.Q2, R232.2
- new net N$287: IC19.Q0, R234.2
- new net N$288: IC20.Q0, R235.2
- new net N$289: IC20.Q7, R239.1
- new net N$290: IC20.Q6, R240.1
- new net N$291: IC20.Q4, R242.1
- new net N$292: LED_STROBE3.Q4, R243.1
- new net N$293: LED_STROBE3.Q5, R244.1
- new net N$294: LED_STROBE3.Q6, R245.1
- new net N$295: LED_STROBE3.Q7, R246.1
- new net N$296: LED_STROBE3.Q3, R247.2
- new net N$297: LED_STROBE3.Q2, R248.2
- new net N$298: LED_STROBE3.Q1, R249.2
- new net N$299: LED_STROBE3.Q0, R250.2
- new net N$300: LED73.A, R227.2
- new net N$301: LED74.A, R228.2
- new net N$302: LED75.A, R229.2
- new net N$303: LED76.A, R230.2
- new net N$304: LED77.A, R231.1
- new net N$305: LED78.A, R232.1
- new net N$306: LED79.A, R233.1
- new net N$307: LED80.A, R234.1
- new net N$308: LED81.A, R235.1
- new net N$309: LED82.A, R236.1
- new net N$310: LED83.A, R237.1
- new net N$311: LED84.A, R238.1
- new net N$312: LED85.A, R239.2
- new net N$313: LED86.A, R240.2
- new net N$314: LED87.A, R241.2
- new net N$315: LED88.A, R242.2
- new net N$316: LED89.A, R243.2
- new net N$317: LED90.A, R244.2
- new net N$318: LED91.A, R245.2
- new net N$319: LED92.A, R246.2
- new net N$320: LED93.A, R247.1
- new net N$321: LED94.A, R248.1
- new net N$322: LED95.A, R249.1
- new net N$323: LED96.A, R250.1
- new net N$324: IC20.Q5, R241.1
- new net N$325: IC20.Q1, R236.2
- new net N$326: IC20.Q2, R237.2
- new net N$327: IC20.Q3, R238.2
- new net N$328: IC19.Q4, R227.1
- new net N$329: IC19.Q6, R229.1
- new net N$330: IC19.Q7, R230.1
- new net N$331: IC19.Q1, R233.2
- new net N$332: IC21.Q5, R252.1
- new net N$333: IC21.Q3, R255.2
- new net N$334: IC21.Q2, R256.2
- new net N$335: IC21.Q0, R258.2
- new net N$336: IC22.Q0, R259.2
- new net N$337: IC22.Q7, R263.1
- new net N$338: IC22.Q6, R264.1
- new net N$339: IC22.Q4, R266.1
- new net N$340: LED_STROBE4.Q4, R267.1
- new net N$341: LED_STROBE4.Q5, R268.1
- new net N$342: LED_STROBE4.Q6, R269.1
- new net N$343: LED_STROBE4.Q7, R270.1
- new net N$344: LED_STROBE4.Q3, R271.2
- new net N$345: LED_STROBE4.Q2, R272.2
- new net N$346: LED_STROBE4.Q1, R273.2
- new net N$347: LED_STROBE4.Q0, R274.2
- new net N$348: LED97.A, R251.2
- new net N$349: LED98.A, R252.2
- new net N$350: LED99.A, R253.2
- new net N$351: LED100.A, R254.2
- new net N$352: LED101.A, R255.1
- new net N$353: LED102.A, R256.1
- new net N$354: LED103.A, R257.1
- new net N$355: LED104.A, R258.1
- new net N$356: LED105.A, R259.1
- new net N$357: LED106.A, R260.1
- new net N$358: LED107.A, R261.1
- new net N$359: LED108.A, R262.1
- new net N$360: LED109.A, R263.2
- new net N$361: LED110.A, R264.2
- new net N$362: LED111.A, R265.2
- new net N$363: LED112.A, R266.2
- new net N$364: LED113.A, R267.2
- new net N$365: LED114.A, R268.2
- new net N$366: LED115.A, R269.2
- new net N$367: LED116.A, R270.2
- new net N$368: LED117.A, R271.1
- new net N$369: LED118.A, R272.1
- new net N$370: LED119.A, R273.1
- new net N$371: LED120.A, R274.1
- new net N$372: IC22.Q5, R265.1
- new net N$373: IC22.Q1, R260.2
- new net N$374: IC22.Q2, R261.2
- new net N$375: IC22.Q3, R262.2
- new net N$376: IC21.Q4, R251.1
- new net N$377: IC21.Q6, R253.1
- new net N$378: IC21.Q7, R254.1
- new net N$379: IC21.Q1, R257.2
- new net N$380: IC23.Q5, R276.1
- new net N$381: IC23.Q3, R279.2
- new net N$382: IC23.Q2, R280.2
- new net N$383: IC23.Q0, R282.2
- new net N$384: IC24.Q0, R283.2
- new net N$385: IC24.Q7, R287.1
- new net N$386: IC24.Q6, R288.1
- new net N$387: IC24.Q4, R290.1
- new net N$388: LED_STROBE5.Q4, R291.1
- new net N$389: LED_STROBE5.Q5, R292.1
- new net N$390: LED_STROBE5.Q6, R293.1
- new net N$391: LED_STROBE5.Q7, R294.1
- new net N$392: LED_STROBE5.Q3, R295.2
- new net N$393: LED_STROBE5.Q2, R296.2
- new net N$394: LED_STROBE5.Q1, R297.2
- new net N$395: LED_STROBE5.Q0, R298.2
- new net N$396: LED121.A, R275.2
- new net N$397: LED122.A, R276.2
- new net N$398: LED123.A, R277.2
- new net N$399: LED124.A, R278.2
- new net N$400: LED125.A, R279.1
- new net N$401: LED126.A, R280.1
- new net N$402: LED127.A, R281.1
- new net N$403: LED128.A, R282.1
- new net N$404: LED129.A, R283.1
- new net N$405: LED130.A, R284.1
- new net N$406: LED131.A, R285.1
- new net N$407: LED132.A, R286.1
- new net N$408: LED133.A, R287.2
- new net N$409: LED134.A, R288.2
- new net N$410: LED135.A, R289.2
- new net N$411: LED136.A, R290.2
- new net N$412: LED137.A, R291.2
- new net N$413: LED138.A, R292.2
- new net N$414: LED139.A, R293.2
- new net N$415: LED140.A, R294.2
- new net N$416: LED141.A, R295.1
- new net N$417: LED142.A, R296.1
- new net N$418: LED143.A, R297.1
- new net N$419: LED144.A, R298.1
- new net N$420: IC24.Q5, R289.1
- new net N$421: IC24.Q1, R284.2
- new net N$422: IC24.Q2, R285.2
- new net N$423: IC24.Q3, R286.2
- new net N$424: IC23.Q4, R275.1
- new net N$425: IC23.Q6, R277.1
- new net N$426: IC23.Q7, R278.1
- new net N$427: IC23.Q1, R281.2
- new net N$428: IC25.Q5, R300.1
- new net N$429: IC25.Q3, R303.2
- new net N$430: IC25.Q2, R304.2
- new net N$431: IC25.Q0, R306.2
- new net N$432: IC26.Q0, R307.2
- new net N$433: IC26.Q7, R311.1
- new net N$434: IC26.Q6, R312.1
- new net N$435: IC26.Q4, R314.1
- new net N$436: LED_STROBE6.Q4, R315.1
- new net N$437: LED_STROBE6.Q5, R316.1
- new net N$438: LED_STROBE6.Q6, R317.1
- new net N$439: LED_STROBE6.Q7, R318.1
- new net N$440: LED_STROBE6.Q3, R319.2
- new net N$441: LED_STROBE6.Q2, R320.2
- new net N$442: LED_STROBE6.Q1, R321.2
- new net N$443: LED_STROBE6.Q0, R322.2
- new net N$444: LED145.A, R299.2
- new net N$445: LED146.A, R300.2
- new net N$446: LED147.A, R301.2
- new net N$447: LED148.A, R302.2
- new net N$448: LED149.A, R303.1
- new net N$449: LED150.A, R304.1
- new net N$450: LED151.A, R305.1
- new net N$451: LED152.A, R306.1
- new net N$452: LED153.A, R307.1
- new net N$453: LED154.A, R308.1
- new net N$454: LED155.A, R309.1
- new net N$455: LED156.A, R310.1
- new net N$456: LED157.A, R311.2
- new net N$457: LED158.A, R312.2
- new net N$458: LED159.A, R313.2
- new net N$459: LED160.A, R314.2
- new net N$460: LED161.A, R315.2
- new net N$461: LED162.A, R316.2
- new net N$462: LED163.A, R317.2
- new net N$463: LED164.A, R318.2
- new net N$464: LED165.A, R319.1
- new net N$465: LED166.A, R320.1
- new net N$466: LED167.A, R321.1
- new net N$467: LED168.A, R322.1
- new net N$468: IC26.Q5, R313.1
- new net N$469: IC26.Q1, R308.2
- new net N$470: IC26.Q2, R309.2
- new net N$471: IC26.Q3, R310.2
- new net N$472: IC25.Q4, R299.1
- new net N$473: IC25.Q6, R301.1
- new net N$474: IC25.Q7, R302.1
- new net N$475: IC25.Q1, R305.2
- new net N$476: IC27.Q5, R324.1
- new net N$477: IC27.Q3, R327.2
- new net N$478: IC27.Q2, R328.2
- new net N$479: IC27.Q0, R330.2
- new net N$480: IC28.Q0, R331.2
- new net N$481: IC28.Q7, R335.1
- new net N$482: IC28.Q6, R336.1
- new net N$483: IC28.Q4, R338.1
- new net N$484: LED_STROBE7.Q4, R339.1
- new net N$485: LED_STROBE7.Q5, R340.1
- new net N$486: LED_STROBE7.Q6, R341.1
- new net N$487: LED_STROBE7.Q7, R342.1
- new net N$488: LED_STROBE7.Q3, R343.2
- new net N$489: LED_STROBE7.Q2, R344.2
- new net N$490: LED_STROBE7.Q1, R345.2
- new net N$491: LED_STROBE7.Q0, R346.2
- new net N$492: LED169.A, R323.2
- new net N$493: LED170.A, R324.2
- new net N$494: LED171.A, R325.2
- new net N$495: LED172.A, R326.2
- new net N$496: LED173.A, R327.1
- new net N$497: LED174.A, R328.1
- new net N$498: LED175.A, R329.1
- new net N$499: LED176.A, R330.1
- new net N$500: LED177.A, R331.1
- new net N$501: LED178.A, R332.1
- new net N$502: LED179.A, R333.1
- new net N$503: LED180.A, R334.1
- new net N$504: LED181.A, R335.2
- new net N$505: LED182.A, R336.2
- new net N$506: LED183.A, R337.2
- new net N$507: LED184.A, R338.2
- new net N$508: LED185.A, R339.2
- new net N$509: LED186.A, R340.2
- new net N$510: LED187.A, R341.2
- new net N$511: LED188.A, R342.2
- new net N$512: LED189.A, R343.1
- new net N$513: LED190.A, R344.1
- new net N$514: LED191.A, R345.1
- new net N$515: LED192.A, R346.1
- new net N$516: IC28.Q5, R337.1
- new net N$517: IC28.Q1, R332.2
- new net N$518: IC28.Q2, R333.2
- new net N$519: IC28.Q3, R334.2
- new net N$520: IC27.Q4, R323.1
- new net N$521: IC27.Q6, R325.1
- new net N$522: IC27.Q7, R326.1
- new net N$523: IC27.Q1, R329.2
- new net N$524: R349.1, VR5.S
- new net N$525: U$22.IN8, U4.QH
- new net N$526: U$22.IN7, U4.QG
- new net N$527: U$22.IN6, U4.QF
- new net N$528: U$22.IN5, U4.QE
- new net N$529: U$22.IN4, U4.QD
- new net N$530: U$22.IN3, U4.QC
- new net N$531: U$22.IN2, U4.QB
- new net N$532: U$22.IN1, U4.QA
- new net N$533: R347.1, U$25.2
- new net N$534: C146.1, IC29A.-IN, R347.2, R348.2, R349.2, R353.2
- new net N$535: R350.1, U$26.2
- new net N$536: R352.1, VR6.S
- new net N$537: C147.1, IC29C.-IN, R350.2, R351.2, R352.2, R354.2
- new net N$538: R357.1, VR7.S
- new net N$539: R355.1, U$27.2
- new net N$540: C150.1, IC29B.+IN, R355.2, R356.2, R357.2, R358.2
- new net N$541: R359.1, U$28.2
- new net N$542: R361.1, VR8.S
- new net N$543: C151.1, IC29D.+IN, R359.2, R360.2, R361.2, R362.2
- net +12V: now also C148.1, IC29P.V+
- net +3V3: now also D1.1, D2.2, D3.1, D4.2, D5.1, D6.2, D7.1, D8.2, IC15.OE, IC15.VCC, IC16.OE, IC16.VCC, IC19.OE, IC19.VCC, IC20.OE, IC20.VCC, IC21.OE, IC21.VCC, IC22.OE, IC22.VCC, IC23.OE, IC23.VCC, IC24.OE, IC24.VCC, IC25.OE, IC25.VCC, IC26.OE, IC26.VCC, IC27.OE, IC27.VCC, IC28.OE, IC28.VCC, LED_STROBE2.OE, LED_STROBE2.VCC, LED_STROBE3.OE, LED_STROBE3.VCC, LED_STROBE4.OE, LED_STROBE4.VCC, LED_STROBE5.OE, LED_STROBE5.VCC, LED_STROBE6.OE, LED_STROBE6.VCC, LED_STROBE7.OE, LED_STROBE7.VCC, U4.VCC
- net +5V: now also U$24G$1.VIN
- net -10V: now also R353.1, R354.1, R358.1, R362.1, VR5.E, VR6.E, VR7.E, VR8.E
- net -12V: now also C149.2, IC29P.V-
- net AIN0+: no longer D2.CATHODE_(DIODE_1),_ANODE_(DIODE_2)
- net AIN0-: no longer D1.CATHODE_(DIODE_1),_ANODE_(DIODE_2)
- net AIN1+: no longer D4.CATHODE_(DIODE_1),_ANODE_(DIODE_2)
- net AIN1-: no longer D3.CATHODE_(DIODE_1),_ANODE_(DIODE_2)
- net AIN2+: no longer D6.CATHODE_(DIODE_1),_ANODE_(DIODE_2)
- net AIN2-: no longer D5.CATHODE_(DIODE_1),_ANODE_(DIODE_2)
- net AIN3+: no longer D8.CATHODE_(DIODE_1),_ANODE_(DIODE_2)
- net AIN3-: no longer D7.CATHODE_(DIODE_1),_ANODE_(DIODE_2)
- net GND: now also C148.2, C149.1, D1.2, D2.1, D3.2, D4.1, D5.2, D6.1, D7.2, D8.1, IC15.GND, IC16.GND, IC19.GND, IC20.GND, IC21.GND, IC22.GND, IC23.GND, IC24.GND, IC25.GND, IC26.GND, IC27.GND, IC28.GND, IC29A.+IN, IC29B.-IN, IC29C.+IN, IC29D.-IN, LED101.C, LED102.C, LED103.C, LED104.C, LED105.C, LED106.C, LED107.C, LED108.C, LED117.C, LED118.C, LED119.C, LED120.C, LED125.C, LED126.C, LED127.C, LED128.C, LED129.C, LED130.C, LED131.C, LED132.C, LED141.C, LED142.C, LED143.C, LED144.C, LED149.C, LED150.C, LED151.C, LED152.C, LED153.C, LED154.C, LED155.C, LED156.C, LED165.C, LED166.C, LED167.C, LED168.C, LED173.C, LED174.C, LED175.C, LED176.C, LED177.C, LED178.C, LED179.C, LED180.C, LED189.C, LED190.C, LED191.C, LED192.C, LED53.C, LED54.C, LED55.C, LED56.C, LED57.C, LED58.C, LED59.C, LED60.C, LED69.C, LED70.C, LED71.C, LED72.C, LED77.C, LED78.C, LED79.C, LED80.C, LED81.C, LED82.C, LED83.C, LED84.C, LED93.C, LED94.C, LED95.C, LED96.C, LED_STROBE2.GND, LED_STROBE3.GND, LED_STROBE4.GND, LED_STROBE5.GND, LED_STROBE6.GND, LED_STROBE7.GND, U$22.COM, U$22.GND, U$24G$1.GND@2, U$25.1, U$25.3, U$26.1, U$26.3, U$27.1, U$27.3, U$28.1, U$28.3, U4.GND, VR5.A, VR6.A, VR7.A, VR8.A; no longer LED1.C, LED13.C, LED14.C, LED15.C, LED16.C, LED17.C, LED18.C, LED19.C, LED2.C, LED20.C, LED25.C, LED26.C, LED27.C, LED28.C, LED3.C, LED37.C, LED38.C, LED39.C, LED4.C, LED40.C, LED41.C, LED42.C, LED43.C, LED44.C
- net LED_CLK: now also IC16.CP, IC20.CP, IC22.CP, IC24.CP, IC26.CP, IC28.CP, LED_STROBE2.CP, LED_STROBE3.CP, LED_STROBE4.CP, LED_STROBE5.CP, LED_STROBE6.CP, LED_STROBE7.CP
- net LED_DATA1: now also IC15.CP, IC16.DATA, IC18.DATA, IC19.CP, IC20.DATA, IC21.CP, IC22.DATA, IC23.CP, IC24.DATA, IC25.CP, IC26.DATA, IC27.CP, IC28.DATA
- net LED_DATA2: no longer IC18.DATA
- net LED_S1: now also IC15.DATA, IC16.QS1, IC17.DATA, IC18.QS1, IC19.DATA, IC20.QS1, IC21.DATA, IC22.QS1, IC23.DATA, IC24.QS1, IC25.DATA, IC26.QS1, IC27.DATA, IC28.QS1
- net LED_S2: now also IC15.QS1, IC17.QS1, IC19.QS1, IC21.QS1, IC23.QS1, IC25.QS1, IC27.QS1, LED_STROBE1.DATA, LED_STROBE2.DATA, LED_STROBE3.DATA, LED_STROBE4.DATA, LED_STROBE5.DATA, LED_STROBE6.DATA, LED_STROBE7.DATA
- net LED_STROBE: now also IC15.STROBE, IC16.STROBE, IC19.STROBE, IC20.STROBE, IC21.STROBE, IC22.STROBE, IC23.STROBE, IC24.STROBE, IC25.STROBE, IC26.STROBE, IC27.STROBE, IC28.STROBE, LED_STROBE2.STROBE, LED_STROBE3.STROBE, LED_STROBE4.STROBE, LED_STROBE5.STROBE, LED_STROBE6.STROBE, LED_STROBE7.STROBE
- net N$144: now also IC15.Q5; no longer IC17.Q5
- net N$145: now also IC15.Q3; no longer IC17.Q3
- net N$146: now also IC15.Q2; no longer IC17.Q2
- net N$147: now also IC15.Q0; no longer IC17.Q0
- net N$148: now also IC16.Q0; no longer IC18.Q0
- net N$149: now also IC16.Q7; no longer IC18.Q7
- net N$150: now also IC16.Q6; no longer IC18.Q6
- net N$151: now also IC16.Q4; no longer IC18.Q4
- net N$226: now also IC16.Q5; no longer IC18.Q5
- net N$227: now also IC16.Q1; no longer IC18.Q1
- net N$228: now also IC16.Q2; no longer IC18.Q2
- net N$229: now also IC16.Q3; no longer IC18.Q3
- net N$230: now also IC15.Q4; no longer IC17.Q4
- net N$231: now also IC15.Q6; no longer IC17.Q6
- net N$232: now also IC15.Q7; no longer IC17.Q7
- net N$233: now also IC15.Q1; no longer IC17.Q1
- net N$235: now also D2.3, D4.3, D6.3, D8.3; no longer D1.ANODE_(DIODE_1), D2.ANODE_(DIODE_1)
- net N$236: now also IC17.Q5, R204.1; no longer D1.CATHODE_(DIODE_2), D2.CATHODE_(DIODE_2)
- net N$237: now also IC17.Q3, R207.2; no longer D3.ANODE_(DIODE_1), D4.ANODE_(DIODE_1)
- net N$238: now also IC17.Q2, R208.2; no longer D3.CATHODE_(DIODE_2), D4.CATHODE_(DIODE_2)
- net N$239: now also IC17.Q0, R210.2; no longer D5.ANODE_(DIODE_1), D6.ANODE_(DIODE_1)
- net N$240: now also IC18.Q0, R211.2; no longer D5.CATHODE_(DIODE_2), D6.CATHODE_(DIODE_2)
- net N$241: now also IC18.Q7, R215.1; no longer D7.ANODE_(DIODE_1), D8.ANODE_(DIODE_1)
- net N$242: now also IC18.Q6, R216.1; no longer D7.CATHODE_(DIODE_2), D8.CATHODE_(DIODE_2)
Other:
- note added: "CV & Pot Controls"
- note removed: "Tactile and CV Controls"

Commit message: schematic has multiplexed LEDs. Need to swap 0805 for 0604s
Parts:
- removed R29: 33R, rcl:R-EU_R0603
- removed U$24: PHOTON_SMD, Particle-Devices:PHOTON_SMD
- removed U4: SN74HC595D, SparkFun-IC-Logic:74HC595D
- added C152, C153: 100n, rcl:C-EUC0603
- added C154: 100n, rcl:C-EUC0805
- added C155, C156, C157, C158, C159, C160, C161, C162, C163, C164, C165, C166, C167, C168, C169, C170, C171, C172: 100nf, rcl:C-EUC0603
- added IC30: 4051D, 40xx:4051D
- added IC31: 4024D, 40xx:4024D
- added IC33: 4017D, 40xx:4017D
- added R363: 2.2k, rcl:R-EU_R0603
- added R364, R368, R369, R370: 33R, rcl:R-EU_R0603
- added R366, R367: 10k, rcl:R-EU_R0603
- C40, C43: device rcl:C-EUC0805 -> rcl:C-EUC0603
- C44: value 0.1u -> 100n; device rcl:C-EUC0805 -> rcl:C-EUC0603
- IC2: value 25AA1024-I_SM -> 24AA1025; device SamacSys_Parts:25AA1024-I_SM -> audioic:24AA1025
- R53: value 10k -> 2.2k
- R56, R59, R60: value 33 -> 33R
- R58: value 33 -> 10k
Connections:
- removed net LED_DATA2: R29.2
- removed net MISO: R56.2, U$1G$2.MISO/SDA_30
- removed net MISO_M: IC2.SO, U$1G$2.SDA_M/MISO_M/MP3_29
- removed net MOSI: R59.2, U$1G$2.MOSI/ADDR1_32
- removed net MOSI_M: IC2.SI, U$1G$2.MOSI_M/MP1_27
- removed net N$136: R29.1, U$1G$5.SDATA_OUT3_52
- removed net SCLK: R58.2, U$1G$2.SCLK/SCL_31
- removed net SCLK_M: IC2.SCK, U$1G$2.SCL_M/SCLK_M/MP2_28
- removed net SS: R60.2, U$1G$2.SS/ADDR0_33
- removed net SS_M: IC2.!CS, R17.1, U$1G$2.SS_M/MP0_26
- new net N$30: R17.1, U$1G$2.SS_M/MP0_26
- new net N$544: IC2.WP, R53.1
- new net N$545: R367.1, U$1G$2.SELFBOOT_34
- new net N$547: R364.1, U$1G$2.SCL_M/MP2_28
- new net N$548: IC30A.X, U$1G$1.AUXADC0_8
- new net N$549: IC2.SCL, R364.2
- new net N$550: R368.1, U$1G$2.SDA_M/MP3_29
- new net N$551: R60.2, U$1G$5.MP6_45
- new net N$552: IC2.SDA, R368.2
- new net N$553: R370.1, U$1G$2.SCLK/SCL_31
- new net N$554: R369.1, U$1G$2.MISO/SDA_30
- new net N$555: IC30A.INH, R58.2
- new net N$556: IC31A.Q4, IC31A.Q5, IC31A.Q6, IC31A.Q7, IC31A.RES
- new net N$557: IC33A.Q8, IC33A.Q9, IC33A.RES
- new net N$558: IC30A.A, IC31A.Q1
- new net N$559: IC30A.B, IC31A.Q2
- new net N$560: IC30A.C, IC31A.Q3
- new net N$562: IC33A.Q6, U$22.IN7
- new net N$563: IC33A.ENA, R366.2
- new net SEL0: R27.2, R59.2
- new net SEL1: R60.1
- new net SEL2: R162.2
- net +3V3: now also C153.2, C154.2, IC30P.VCC, IC30P.VEE, R363.2, R367.2, R58.1; no longer C44.1, IC2.!HOLD, IC2.VCC, R17.2, U$1G$2.SELFBOOT_34, U4.VCC
- net +5V: now also C152.1, C155.1, C156.1, C157.1, C158.1, C159.1, C160.1, C161.1, C162.1, C163.1, C164.1, C165.1, C166.1, C167.1, C168.1, C169.1, C170.1, C171.1, C172.1, C44.1, IC31P.VDD, IC33P.VDD, R366.1; no longer U$24G$1.VIN
- net CV0: now also IC30A.X0; no longer U$1G$1.AUXADC0_8
- net CV1: now also IC30A.X1; no longer U$1G$1.AUXADC1_9
- net CV2: now also IC30A.X2; no longer U$1G$1.AUXADC2_10
- net CV3: now also IC30A.X3; no longer U$1G$1.AUXADC3_11
- net CV4: now also IC30A.X4
- net CV5: now also IC30A.X5
- net CV6: now also IC30A.X6
- net CV7: now also IC30A.X7
- net ENCODER0_0: now also U$1G$1.AUXADC1_9; no longer U$1G$5.MP6_45
- net ENCODER0_1: now also U$1G$1.AUXADC2_10; no longer R162.2
- net ENCODER1_0: now also U$1G$1.AUXADC3_11; no longer U$1G$4.LRCLK_IN1/MP11_61
- net ENCODER1_1: now also U$1G$1.AUXADC4_12; no longer U$1G$4.LRCLK_IN3/MP13_69
- net GND: now also C152.2, C153.1, C154.1, C155.2, C156.2, C157.2, C158.2, C159.2, C160.2, C161.2, C162.2, C163.2, C164.2, C165.2, C166.2, C167.2, C168.2, C169.2, C170.2, C171.2, C172.2, IC2.A0, IC2.A1, IC2.A2*, IC30P.GND, IC31P.VSS, IC33P.VSS, R17.2, U$1G$2.MOSI/ADDR1_32, U$1G$2.SS/ADDR0_33; no longer LED10.C, LED101.C, LED102.C, LED103.C, LED104.C, LED105.C, LED106.C, LED107.C, LED108.C, LED11.C, LED117.C, LED118.C, LED119.C, LED12.C, LED120.C, LED125.C, LED126.C, LED127.C, LED128.C, LED129.C, LED130.C, LED131.C, LED132.C, LED141.C, LED142.C, LED143.C, LED144.C, LED149.C, LED150.C, LED151.C, LED152.C, LED153.C, LED154.C, LED155.C, LED156.C, LED165.C, LED166.C, LED167.C, LED168.C, LED173.C, LED174.C, LED175.C, LED176.C, LED177.C, LED178.C, LED179.C, LED180.C, LED189.C, LED190.C, LED191.C, LED192.C, LED21.C, LED22.C, LED23.C, LED24.C, LED29.C, LED30.C, LED31.C, LED32.C, LED33.C, LED34.C, LED35.C, LED36.C, LED45.C, LED46.C, LED47.C, LED48.C, LED5.C, LED53.C, LED54.C, LED55.C, LED56.C, LED57.C, LED58.C, LED59.C, LED6.C, LED60.C, LED69.C, LED7.C, LED70.C, LED71.C, LED72.C, LED77.C, LED78.C, LED79.C, LED8.C, LED80.C, LED81.C, LED82.C, LED83.C, LED84.C, LED9.C, LED93.C, LED94.C, LED95.C, LED96.C, U$24G$1.GND@2, U4.GND
- net LED_CLK: now also IC13.CP, IC15.CP, IC17.CP, IC19.CP, IC21.CP, IC23.CP, IC25.CP, IC27.CP
- net LED_DATA1: no longer IC13.CP, IC15.CP, IC17.CP, IC19.CP, IC21.CP, IC23.CP, IC25.CP, IC27.CP
- net LED_ROW_1: now also LED10.C, LED11.C, LED12.C, LED21.C, LED22.C, LED23.C, LED24.C, LED5.C, LED6.C, LED7.C, LED8.C, LED9.C; no longer LED100.C, LED109.C, LED110.C, LED111.C, LED112.C, LED113.C, LED114.C, LED115.C, LED116.C, LED121.C, LED122.C, LED123.C, LED124.C, LED133.C, LED134.C, LED135.C, LED136.C, LED137.C, LED138.C, LED139.C, LED140.C, LED145.C, LED146.C, LED147.C, LED148.C, LED157.C, LED158.C, LED159.C, LED160.C, LED161.C, LED162.C, LED163.C, LED164.C, LED169.C, LED170.C, LED171.C, LED172.C, LED181.C, LED182.C, LED183.C, LED184.C, LED185.C, LED186.C, LED187.C, LED188.C, LED25.C, LED26.C, LED27.C, LED28.C, LED37.C, LED38.C, LED39.C, LED40.C, LED41.C, LED42.C, LED43.C, LED44.C, LED49.C, LED50.C, LED51.C, LED52.C, LED61.C, LED62.C, LED63.C, LED64.C, LED65.C, LED66.C, LED67.C, LED68.C, LED73.C, LED74.C, LED75.C, LED76.C, LED85.C, LED86.C, LED87.C, LED88.C, LED89.C, LED90.C, LED91.C, LED92.C, LED97.C, LED98.C, LED99.C
- net LED_ROW_2: now also LED25.C, LED26.C, LED27.C, LED28.C, LED29.C, LED30.C, LED31.C, LED32.C, LED33.C, LED34.C, LED35.C, LED36.C, LED37.C, LED38.C, LED39.C, LED40.C, LED41.C, LED42.C, LED43.C, LED44.C, LED45.C, LED46.C, LED47.C, LED48.C
- net LED_ROW_3: now also LED49.C, LED50.C, LED51.C, LED52.C, LED53.C, LED54.C, LED55.C, LED56.C, LED57.C, LED58.C, LED59.C, LED60.C, LED61.C, LED62.C, LED63.C, LED64.C, LED65.C, LED66.C, LED67.C, LED68.C, LED69.C, LED70.C, LED71.C, LED72.C
- net LED_ROW_4: now also LED73.C, LED74.C, LED75.C, LED76.C, LED77.C, LED78.C, LED79.C, LED80.C, LED81.C, LED82.C, LED83.C, LED84.C, LED85.C, LED86.C, LED87.C, LED88.C, LED89.C, LED90.C, LED91.C, LED92.C, LED93.C, LED94.C, LED95.C, LED96.C
- net LED_ROW_5: now also LED100.C, LED101.C, LED102.C, LED103.C, LED104.C, LED105.C, LED106.C, LED107.C, LED108.C, LED109.C, LED110.C, LED111.C, LED112.C, LED113.C, LED114.C, LED115.C, LED116.C, LED117.C, LED118.C, LED119.C, LED120.C, LED97.C, LED98.C, LED99.C
- net LED_ROW_6: now also LED121.C, LED122.C, LED123.C, LED124.C, LED125.C, LED126.C, LED127.C, LED128.C, LED129.C, LED130.C, LED131.C, LED132.C, LED133.C, LED134.C, LED135.C, LED136.C, LED137.C, LED138.C, LED139.C, LED140.C, LED141.C, LED142.C, LED143.C, LED144.C
- net LED_ROW_7: now also LED145.C, LED146.C, LED147.C, LED148.C, LED149.C, LED150.C, LED151.C, LED152.C, LED153.C, LED154.C, LED155.C, LED156.C, LED157.C, LED158.C, LED159.C, LED160.C, LED161.C, LED162.C, LED163.C, LED164.C, LED165.C, LED166.C, LED167.C, LED168.C
- net LED_ROW_8: now also LED169.C, LED170.C, LED171.C, LED172.C, LED181.C, LED182.C, LED183.C, LED184.C, LED185.C, LED186.C, LED187.C, LED188.C
- net LED_STROBE: now also IC31A.CLK, IC33A.CLK
- net N$138: now also U$1G$4.LRCLK_IN1/MP11_61; no longer U$1G$5.LRCLK_OUT3/MP9_50
- net N$31: now also U$1G$2.MP1_27; no longer X1-8.KL
- net N$32: now also R370.2, X1-1.KL; no longer R60.1, X1-9.KL
- net N$37: now also R369.2, X1-3.KL; no longer R56.1, X1-5.KL
- net N$39: now also R56.1, U$1G$5.LRCLK_OUT3/MP9_50; no longer R58.1, X1-7.KL
- net N$525: now also IC33A.Q7; no longer U4.QH
- net N$526: now also LED173.C, LED174.C, LED175.C, LED176.C, LED177.C, LED178.C, LED179.C, LED180.C, LED189.C, LED190.C, LED191.C, LED192.C; no longer U$22.IN7, U4.QG
- net N$527: now also IC33A.Q5; no longer U4.QF
- net N$528: now also IC33A.Q4; no longer U4.QE
- net N$529: now also IC33A.Q3; no longer U4.QD
- net N$530: now also IC33A.Q2; no longer U4.QC
- net N$531: now also IC33A.Q1; no longer U4.QB
- net N$532: now also IC33A.Q0; no longer U4.QA
- net N$7: now also IC2.VCC, R363.1; no longer IC2.!WP, R53.1
- net SW1: now also R56.2; no longer R27.2
Other:
- note added: "I2C EEPROM"
- note added: "LED Supply Decoupling"
- note removed: "SPI EEPROM"
