File: DSPBoard.sch (EAGLE design)
At the start: 825 parts, among them IC1 AD1939WBSTZ, IC10 LM833D, IC11 LM833D, IC12 TL074D, IC13 CD74HC4094M96, IC14 CD74HC4094M96, IC15 CD74HC4094M96, IC16 CD74HC4094M96, IC17 CD74HC4094M96, IC18 CD74HC4094M96, IC19 CD74HC4094M96, IC2 24AA1025, IC20 CD74HC4094M96, IC21 CD74HC4094M96, IC22 CD74HC4094M96, IC23 CD74HC4094M96, IC24 CD74HC4094M96, IC25 CD74HC4094M96, IC26 CD74HC4094M96, IC27 CD74HC4094M96, IC28 CD74HC4094M96, IC29 TL074D, IC3 LM4040B10DBZ, IC30 4051D, IC31 4024D, IC33 4017D, IC4 LM833D, IC5 LM833D, IC6 LM833D, IC7 LM833D, IC8 LM833D, IC9 LM833D, U1 LM11173.3NOPB, U2 PEC11R-4315F-N0012, U3 PEC11R-4315F-N0012, X1 2510-, Y1 12.288MHz

Commit message: update
Parts:
- removed R53: 2.2k, rcl:R-EU_R0603
- C1, C100, C101, C102, C103, C104, C105, C106, C107, C108, C109, C110, C111, C112, C113, C114, C115, C116, C117, C118, C119, C120, C121, C122, C123, C124, C125, C126, C127, C128, C129, C130, C131, C132, C133, C134, C135, C137, C138, C139, C140, C141, C142, C143, C144, C145, C146, C147, C148, C149, C150, C151, C154, C17, C18, C24, C25, C26, C27, C28, C29, C30, C31, C32, C33, C34, C36, C37, C38, C41, C42, C45, C46, C47, C48, C49, C5, C51, C52, C53, C55, C56, C57, C58, C59, C6, C60, C62, C63, C64, C66, C67, C68, C69, C70, C71, C73, C74, C75, C77, C78, C79, C80, C81, C82, C83, C84, C85, C86, C87, C88, C89, C90, C91, C92, C93, C94, C95, C97, C99: device rcl:C-EUC0805 -> rcl:C-EUC0603
- C136, C39, C54, C65, C76: device rcl:CPOL-EU140CLH-0810 -> rcl:CPOL-EUD
- C35, C50, C61, C72: device rcl:CPOL-EU140CLH-1014 -> rcl:CPOL-EUD
- R10, R100, R101, R102, R103, R104, R105, R106, R107, R108, R109, R11, R110, R111, R112, R113, R114, R115, R116, R117, R118, R119, R120, R121, R122, R123, R124, R125, R126, R127, R128, R129, R130, R131, R132, R133, R134, R136, R137, R138, R139, R14, R140, R141, R143, R144, R145, R146, R147, R148, R149, R15, R150, R151, R152, R153, R154, R155, R156, R157, R158, R159, R16, R160, R161, R163, R164, R165, R166, R167, R168, R169, R170, R171, R172, R173, R174, R175, R176, R177, R178, R179, R180, R181, R182, R183, R184, R185, R186, R187, R188, R189, R190, R191, R192, R193, R194, R195, R196, R197, R198, R199, R2, R200, R201, R202, R203, R204, R205, R206, R207, R208, R209, R21, R210, R211, R212, R213, R214, R215, R216, R217, R218, R219, R22, R220, R221, R222, R223, R224, R225, R226, R227, R228, R229, R230, R231, R232, R233, R234, R235, R236, R237, R238, R239, R240, R241, R242, R243, R244, R245, R246, R247, R248, R249, R250, R251, R252, R253, R254, R255, R256, R257, R258, R259, R260, R261, R262, R263, R264, R265, R266, R267, R268, R269, R270, R271, R272, R273, R274, R275, R276, R277, R278, R279, R28, R280, R281, R282, R283, R284, R285, R286, R287, R288, R289, R290, R291, R292, R293, R294, R295, R296, R297, R298, R299, R3, R30, R300, R301, R302, R303, R304, R305, R306, R307, R308, R309, R31, R310, R311, R312, R313, R314, R315, R316, R317, R318, R319, R32, R320, R321, R322, R323, R324, R325, R326, R327, R328, R329, R33, R330, R331, R332, R333, R334, R335, R336, R337, R338, R339, R34, R340, R341, R342, R343, R344, R345, R346, R347, R348, R349, R35, R350, R351, R352, R353, R354, R355, R356, R357, R358, R359, R36, R360, R361, R362, R37, R38, R39, R4, R40, R41, R42, R43, R44, R45, R46, R47, R48, R49, R5, R50, R51, R54, R55, R57, R6, R61, R62, R63, R64, R65, R66, R67, R68, R69, R7, R70, R71, R72, R73, R74, R75, R76, R77, R78, R79, R8, R80, R81, R82, R83, R84, R85, R86, R87, R88, R89, R9, R90, R91, R92, R93, R94, R95, R96, R97, R98, R99: device rcl:R-EU_R0805 -> rcl:R-EU_R0603
Connections:
- removed net N$544: IC2.WP, R53.1
- net +3V3: no longer R53.2
- net GND: now also IC2.WP

Commit message: removed LEDS
Parts:
- removed C155, C156, C157, C158, C159, C160, C161, C162, C163, C164, C165, C166, C167, C168, C169, C170, C171, C172: 100nf, rcl:C-EUC0603
- removed IC13, IC14, IC15, IC16, IC17, IC18, IC19, IC20, IC21, IC22, IC23, IC24, IC25, IC26, IC27, IC28, LED_STROBE, LED_STROBE1, LED_STROBE2, LED_STROBE3, LED_STROBE4, LED_STROBE5, LED_STROBE6, LED_STROBE7: CD74HC4094M96, CD74HC4094M96:CD74HC4094M96
- removed LED1, LED10, LED100, LED101, LED102, LED103, LED104, LED105, LED106, LED107, LED108, LED109, LED11, LED110, LED111, LED112, LED113, LED114, LED115, LED116, LED117, LED118, LED119, LED12, LED120, LED121, LED122, LED123, LED124, LED125, LED126, LED127, LED128, LED129, LED13, LED130, LED131, LED132, LED133, LED134, LED135, LED136, LED137, LED138, LED139, LED14, LED140, LED141, LED142, LED143, LED144, LED145, LED146, LED147, LED148, LED149, LED15, LED150, LED151, LED152, LED153, LED154, LED155, LED156, LED157, LED158, LED159, LED16, LED160, LED161, LED162, LED163, LED164, LED165, LED166, LED167, LED168, LED169, LED17, LED170, LED171, LED172, LED173, LED174, LED175, LED176, LED177, LED178, LED179, LED18, LED180, LED181, LED182, LED183, LED184, LED185, LED186, LED187, LED188, LED189, LED19, LED190, LED191, LED192, LED2, LED20, LED21, LED22, LED23, LED24, LED25, LED26, LED27, LED28, LED29, LED3, LED30, LED31, LED32, LED33, LED34, LED35, LED36, LED37, LED38, LED39, LED4, LED40, LED41, LED42, LED43, LED44, LED45, LED46, LED47, LED48, LED49, LED5, LED50, LED51, LED52, LED53, LED54, LED55, LED56, LED57, LED58, LED59, LED6, LED60, LED61, LED62, LED63, LED64, LED65, LED66, LED67, LED68, LED69, LED7, LED70, LED71, LED72, LED73, LED74, LED75, LED76, LED77, LED78, LED79, LED8, LED80, LED81, LED82, LED83, LED84, LED85, LED86, LED87, LED88, LED89, LED9, LED90, LED91, LED92, LED93, LED94, LED95, LED96, LED97, LED98, LED99: (no value), led:LEDCHIPLED_0805
- removed R154, R155, R156, R157, R158, R159, R160, R161, R163, R164, R165, R166, R167, R168, R169, R170, R171, R172, R173, R174, R175, R176, R181, R182, R183, R184, R185, R186, R187, R188, R189, R190, R195, R196, R197, R198, R199, R200, R201, R202, R203, R204, R205, R206, R207, R208, R209, R210, R211, R212, R213, R214, R219, R220, R221, R222, R223, R224, R225, R226, R227, R228, R229, R230, R231, R232, R233, R234, R235, R236, R237, R238, R243, R244, R245, R246, R247, R248, R249, R250, R251, R252, R253, R254, R255, R256, R257, R258, R259, R260, R261, R262, R267, R268, R269, R270, R271, R272, R273, R274, R275, R276, R277, R278, R279, R280, R281, R282, R283, R284, R285, R286, R291, R292, R293, R294, R295, R296, R297, R298, R299, R300, R301, R302, R303, R304, R305, R306, R307, R308, R309, R310, R315, R316, R317, R318, R319, R320, R321, R322, R323, R324, R325, R326, R327, R328, R329, R330, R331, R332, R333, R334, R339, R340, R341, R342, R343, R344, R345, R346: 470R, rcl:R-EU_R0603
- removed R177, R178, R179, R180, R191, R192, R193, R194, R215, R216, R217, R218, R239, R240, R241, R242, R263, R264, R265, R266, R287, R288, R289, R290, R311, R312, R313, R314, R335, R336, R337, R338: 470, rcl:R-EU_R0603
- added U$24: PHOTON_SMD, Particle-Devices:PHOTON_SMD
Connections:
- removed net LED_S1: IC13.DATA, IC14.QS1, IC15.DATA, IC16.QS1, IC17.DATA, IC18.QS1, IC19.DATA, IC20.QS1, IC21.DATA, IC22.QS1, IC23.DATA, IC24.QS1, IC25.DATA, IC26.QS1, IC27.DATA, IC28.QS1
- removed net LED_S2: IC13.QS1, IC15.QS1, IC17.QS1, IC19.QS1, IC21.QS1, IC23.QS1, IC25.QS1, IC27.QS1, LED_STROBE.DATA, LED_STROBE1.DATA, LED_STROBE2.DATA, LED_STROBE3.DATA, LED_STROBE4.DATA, LED_STROBE5.DATA, LED_STROBE6.DATA, LED_STROBE7.DATA
- removed net N$123: IC14.Q5, R179.1
- removed net N$126: IC14.Q1, R174.2
- removed net N$132: IC14.Q2, R175.2
- removed net N$134: IC14.Q3, R176.2
- removed net N$135: IC13.Q4, R165.1
- removed net N$137: IC13.Q6, R167.1
- removed net N$142: IC13.Q7, R168.1
- removed net N$143: IC13.Q1, R171.2
- removed net N$144: IC15.Q5, R155.1
- removed net N$145: IC15.Q3, R158.2
- removed net N$146: IC15.Q2, R159.2
- removed net N$147: IC15.Q0, R161.2
- removed net N$148: IC16.Q0, R163.2
- removed net N$149: IC16.Q7, R191.1
- removed net N$150: IC16.Q6, R192.1
- removed net N$151: IC16.Q4, R194.1
- removed net N$152: LED_STROBE1.Q4, R195.1
- removed net N$153: LED_STROBE1.Q5, R196.1
- removed net N$154: LED_STROBE1.Q6, R197.1
- removed net N$155: LED_STROBE1.Q7, R198.1
- removed net N$156: LED_STROBE1.Q3, R199.2
- removed net N$157: LED_STROBE1.Q2, R200.2
- removed net N$158: LED_STROBE1.Q1, R201.2
- removed net N$159: LED_STROBE1.Q0, R202.2
- removed net N$160: LED25.A, R154.2
- removed net N$161: LED26.A, R155.2
- removed net N$163: LED27.A, R156.2
- removed net N$164: LED28.A, R157.2
- removed net N$165: IC13.Q5, R166.1
- removed net N$166: LED29.A, R158.1
- removed net N$167: LED30.A, R159.1
- removed net N$168: IC13.Q3, R169.2
- removed net N$169: IC13.Q2, R170.2
- removed net N$170: LED31.A, R160.1
- removed net N$171: IC13.Q0, R172.2
- removed net N$172: IC14.Q0, R173.2
- removed net N$173: LED32.A, R161.1
- removed net N$174: LED33.A, R163.1
- removed net N$175: LED34.A, R164.1
- removed net N$176: IC14.Q7, R177.1
- removed net N$177: IC14.Q6, R178.1
- removed net N$178: LED35.A, R189.1
- removed net N$179: IC14.Q4, R180.1
- removed net N$180: LED_STROBE.Q4, R181.1
- removed net N$181: LED_STROBE.Q5, R182.1
- removed net N$182: LED_STROBE.Q6, R183.1
- removed net N$183: LED_STROBE.Q7, R184.1
- removed net N$184: LED_STROBE.Q3, R185.2
- removed net N$185: LED_STROBE.Q2, R186.2
- removed net N$186: LED_STROBE.Q1, R187.2
- removed net N$187: LED_STROBE.Q0, R188.2
- removed net N$188: LED1.A, R165.2
- removed net N$189: LED2.A, R166.2
- removed net N$190: LED3.A, R167.2
- removed net N$191: LED4.A, R168.2
- removed net N$192: LED5.A, R169.1
- removed net N$193: LED6.A, R170.1
- removed net N$194: LED7.A, R171.1
- removed net N$195: LED8.A, R172.1
- removed net N$196: LED9.A, R173.1
- removed net N$197: LED10.A, R174.1
- removed net N$198: LED11.A, R175.1
- removed net N$199: LED12.A, R176.1
- removed net N$200: LED13.A, R177.2
- removed net N$201: LED14.A, R178.2
- removed net N$202: LED15.A, R179.2
- removed net N$203: LED16.A, R180.2
- removed net N$204: LED17.A, R181.2
- removed net N$205: LED18.A, R182.2
- removed net N$206: LED19.A, R183.2
- removed net N$207: LED20.A, R184.2
- removed net N$208: LED21.A, R185.1
- removed net N$209: LED22.A, R186.1
- removed net N$210: LED23.A, R187.1
- removed net N$211: LED24.A, R188.1
- removed net N$213: LED36.A, R190.1
- removed net N$214: LED37.A, R191.2
- removed net N$215: LED38.A, R192.2
- removed net N$216: LED39.A, R193.2
- removed net N$217: LED40.A, R194.2
- removed net N$218: LED41.A, R195.2
- removed net N$219: LED42.A, R196.2
- removed net N$220: LED43.A, R197.2
- removed net N$221: LED44.A, R198.2
- removed net N$222: LED45.A, R199.1
- removed net N$223: LED46.A, R200.1
- removed net N$224: LED47.A, R201.1
- removed net N$225: LED48.A, R202.1
- removed net N$226: IC16.Q5, R193.1
- removed net N$227: IC16.Q1, R164.2
- removed net N$228: IC16.Q2, R189.2
- removed net N$229: IC16.Q3, R190.2
- removed net N$230: IC15.Q4, R154.1
- removed net N$231: IC15.Q6, R156.1
- removed net N$232: IC15.Q7, R157.1
- removed net N$233: IC15.Q1, R160.2
- removed net N$236: IC17.Q5, R204.1
- removed net N$237: IC17.Q3, R207.2
- removed net N$238: IC17.Q2, R208.2
- removed net N$239: IC17.Q0, R210.2
- removed net N$240: IC18.Q0, R211.2
- removed net N$241: IC18.Q7, R215.1
- removed net N$242: IC18.Q6, R216.1
- removed net N$243: IC18.Q4, R218.1
- removed net N$244: LED_STROBE2.Q4, R219.1
- removed net N$245: LED_STROBE2.Q5, R220.1
- removed net N$246: LED_STROBE2.Q6, R221.1
- removed net N$247: LED_STROBE2.Q7, R222.1
- removed net N$248: LED_STROBE2.Q3, R223.2
- removed net N$249: LED_STROBE2.Q2, R224.2
- removed net N$250: LED_STROBE2.Q1, R225.2
- removed net N$251: LED_STROBE2.Q0, R226.2
- removed net N$252: LED49.A, R203.2
- removed net N$253: LED50.A, R204.2
- removed net N$254: LED51.A, R205.2
- removed net N$255: LED52.A, R206.2
- removed net N$256: LED53.A, R207.1
- removed net N$257: LED54.A, R208.1
- removed net N$258: LED55.A, R209.1
- removed net N$259: LED56.A, R210.1
- removed net N$260: LED57.A, R211.1
- removed net N$261: LED58.A, R212.1
- removed net N$262: LED59.A, R213.1
- removed net N$263: LED60.A, R214.1
- removed net N$264: LED61.A, R215.2
- removed net N$265: LED62.A, R216.2
- removed net N$266: LED63.A, R217.2
- removed net N$267: LED64.A, R218.2
- removed net N$268: LED65.A, R219.2
- removed net N$269: LED66.A, R220.2
- removed net N$270: LED67.A, R221.2
- removed net N$271: LED68.A, R222.2
- removed net N$272: LED69.A, R223.1
- removed net N$273: LED70.A, R224.1
- removed net N$274: LED71.A, R225.1
- removed net N$275: LED72.A, R226.1
- removed net N$276: IC18.Q5, R217.1
- removed net N$277: IC18.Q1, R212.2
- removed net N$278: IC18.Q2, R213.2
- removed net N$279: IC18.Q3, R214.2
- removed net N$280: IC17.Q4, R203.1
- removed net N$281: IC17.Q6, R205.1
- removed net N$282: IC17.Q7, R206.1
- removed net N$283: IC17.Q1, R209.2
- removed net N$284: IC19.Q5, R228.1
- removed net N$285: IC19.Q3, R231.2
- removed net N$286: IC19.Q2, R232.2
- removed net N$287: IC19.Q0, R234.2
- removed net N$288: IC20.Q0, R235.2
- removed net N$289: IC20.Q7, R239.1
- removed net N$290: IC20.Q6, R240.1
- removed net N$291: IC20.Q4, R242.1
- removed net N$292: LED_STROBE3.Q4, R243.1
- removed net N$293: LED_STROBE3.Q5, R244.1
- removed net N$294: LED_STROBE3.Q6, R245.1
- removed net N$295: LED_STROBE3.Q7, R246.1
- removed net N$296: LED_STROBE3.Q3, R247.2
- removed net N$297: LED_STROBE3.Q2, R248.2
- removed net N$298: LED_STROBE3.Q1, R249.2
- removed net N$299: LED_STROBE3.Q0, R250.2
- removed net N$300: LED73.A, R227.2
- removed net N$301: LED74.A, R228.2
- removed net N$302: LED75.A, R229.2
- removed net N$303: LED76.A, R230.2
- removed net N$304: LED77.A, R231.1
- removed net N$305: LED78.A, R232.1
- removed net N$306: LED79.A, R233.1
- removed net N$307: LED80.A, R234.1
- removed net N$308: LED81.A, R235.1
- removed net N$309: LED82.A, R236.1
- removed net N$310: LED83.A, R237.1
- removed net N$311: LED84.A, R238.1
- removed net N$312: LED85.A, R239.2
- removed net N$313: LED86.A, R240.2
- removed net N$314: LED87.A, R241.2
- removed net N$315: LED88.A, R242.2
- removed net N$316: LED89.A, R243.2
- removed net N$317: LED90.A, R244.2
- removed net N$318: LED91.A, R245.2
- removed net N$319: LED92.A, R246.2
- removed net N$320: LED93.A, R247.1
- removed net N$321: LED94.A, R248.1
- removed net N$322: LED95.A, R249.1
- removed net N$323: LED96.A, R250.1
- removed net N$324: IC20.Q5, R241.1
- removed net N$325: IC20.Q1, R236.2
- removed net N$326: IC20.Q2, R237.2
- removed net N$327: IC20.Q3, R238.2
- removed net N$328: IC19.Q4, R227.1
- removed net N$329: IC19.Q6, R229.1
- removed net N$330: IC19.Q7, R230.1
- removed net N$331: IC19.Q1, R233.2
- removed net N$332: IC21.Q5, R252.1
- removed net N$333: IC21.Q3, R255.2
- removed net N$334: IC21.Q2, R256.2
- removed net N$335: IC21.Q0, R258.2
- removed net N$336: IC22.Q0, R259.2
- removed net N$337: IC22.Q7, R263.1
- removed net N$338: IC22.Q6, R264.1
- removed net N$339: IC22.Q4, R266.1
- removed net N$340: LED_STROBE4.Q4, R267.1
- removed net N$341: LED_STROBE4.Q5, R268.1
- removed net N$342: LED_STROBE4.Q6, R269.1
- removed net N$343: LED_STROBE4.Q7, R270.1
- removed net N$344: LED_STROBE4.Q3, R271.2
- removed net N$345: LED_STROBE4.Q2, R272.2
- removed net N$346: LED_STROBE4.Q1, R273.2
- removed net N$347: LED_STROBE4.Q0, R274.2
- removed net N$348: LED97.A, R251.2
- removed net N$349: LED98.A, R252.2
- removed net N$350: LED99.A, R253.2
- removed net N$351: LED100.A, R254.2
- removed net N$352: LED101.A, R255.1
- removed net N$353: LED102.A, R256.1
- removed net N$354: LED103.A, R257.1
- removed net N$355: LED104.A, R258.1
- removed net N$356: LED105.A, R259.1
- removed net N$357: LED106.A, R260.1
- removed net N$358: LED107.A, R261.1
- removed net N$359: LED108.A, R262.1
- removed net N$360: LED109.A, R263.2
- removed net N$361: LED110.A, R264.2
- removed net N$362: LED111.A, R265.2
- removed net N$363: LED112.A, R266.2
- removed net N$364: LED113.A, R267.2
- removed net N$365: LED114.A, R268.2
- removed net N$366: LED115.A, R269.2
- removed net N$367: LED116.A, R270.2
- removed net N$368: LED117.A, R271.1
- removed net N$369: LED118.A, R272.1
- removed net N$370: LED119.A, R273.1
- removed net N$371: LED120.A, R274.1
- removed net N$372: IC22.Q5, R265.1
- removed net N$373: IC22.Q1, R260.2
- removed net N$374: IC22.Q2, R261.2
- removed net N$375: IC22.Q3, R262.2
- removed net N$376: IC21.Q4, R251.1
- removed net N$377: IC21.Q6, R253.1
- removed net N$378: IC21.Q7, R254.1
- removed net N$379: IC21.Q1, R257.2
- removed net N$380: IC23.Q5, R276.1
- removed net N$381: IC23.Q3, R279.2
- removed net N$382: IC23.Q2, R280.2
- removed net N$383: IC23.Q0, R282.2
- removed net N$384: IC24.Q0, R283.2
- removed net N$385: IC24.Q7, R287.1
- removed net N$386: IC24.Q6, R288.1
- removed net N$387: IC24.Q4, R290.1
- removed net N$388: LED_STROBE5.Q4, R291.1
- removed net N$389: LED_STROBE5.Q5, R292.1
- removed net N$390: LED_STROBE5.Q6, R293.1
- removed net N$391: LED_STROBE5.Q7, R294.1
- removed net N$392: LED_STROBE5.Q3, R295.2
- removed net N$393: LED_STROBE5.Q2, R296.2
- removed net N$394: LED_STROBE5.Q1, R297.2
- removed net N$395: LED_STROBE5.Q0, R298.2
- removed net N$396: LED121.A, R275.2
- removed net N$397: LED122.A, R276.2
- removed net N$398: LED123.A, R277.2
- removed net N$399: LED124.A, R278.2
- removed net N$400: LED125.A, R279.1
- removed net N$401: LED126.A, R280.1
- removed net N$402: LED127.A, R281.1
- removed net N$403: LED128.A, R282.1
- removed net N$404: LED129.A, R283.1
- removed net N$405: LED130.A, R284.1
- removed net N$406: LED131.A, R285.1
- removed net N$407: LED132.A, R286.1
- removed net N$408: LED133.A, R287.2
- removed net N$409: LED134.A, R288.2
- removed net N$410: LED135.A, R289.2
- removed net N$411: LED136.A, R290.2
- removed net N$412: LED137.A, R291.2
- removed net N$413: LED138.A, R292.2
- removed net N$414: LED139.A, R293.2
- removed net N$415: LED140.A, R294.2
- removed net N$416: LED141.A, R295.1
- removed net N$417: LED142.A, R296.1
- removed net N$418: LED143.A, R297.1
- removed net N$419: LED144.A, R298.1
- removed net N$420: IC24.Q5, R289.1
- removed net N$421: IC24.Q1, R284.2
- removed net N$422: IC24.Q2, R285.2
- removed net N$423: IC24.Q3, R286.2
- removed net N$424: IC23.Q4, R275.1
- removed net N$425: IC23.Q6, R277.1
- removed net N$426: IC23.Q7, R278.1
- removed net N$427: IC23.Q1, R281.2
- removed net N$428: IC25.Q5, R300.1
- removed net N$429: IC25.Q3, R303.2
- removed net N$430: IC25.Q2, R304.2
- removed net N$431: IC25.Q0, R306.2
- removed net N$432: IC26.Q0, R307.2
- removed net N$433: IC26.Q7, R311.1
- removed net N$434: IC26.Q6, R312.1
- removed net N$435: IC26.Q4, R314.1
- removed net N$436: LED_STROBE6.Q4, R315.1
- removed net N$437: LED_STROBE6.Q5, R316.1
- removed net N$438: LED_STROBE6.Q6, R317.1
- removed net N$439: LED_STROBE6.Q7, R318.1
- removed net N$440: LED_STROBE6.Q3, R319.2
- removed net N$441: LED_STROBE6.Q2, R320.2
- removed net N$442: LED_STROBE6.Q1, R321.2
- removed net N$443: LED_STROBE6.Q0, R322.2
- removed net N$444: LED145.A, R299.2
- removed net N$445: LED146.A, R300.2
- removed net N$446: LED147.A, R301.2
- removed net N$447: LED148.A, R302.2
- removed net N$448: LED149.A, R303.1
- removed net N$449: LED150.A, R304.1
- removed net N$450: LED151.A, R305.1
- removed net N$451: LED152.A, R306.1
- removed net N$452: LED153.A, R307.1
- removed net N$453: LED154.A, R308.1
- removed net N$454: LED155.A, R309.1
- removed net N$455: LED156.A, R310.1
- removed net N$456: LED157.A, R311.2
- removed net N$457: LED158.A, R312.2
- removed net N$458: LED159.A, R313.2
- removed net N$459: LED160.A, R314.2
- removed net N$460: LED161.A, R315.2
- removed net N$461: LED162.A, R316.2
- removed net N$462: LED163.A, R317.2
- removed net N$463: LED164.A, R318.2
- removed net N$464: LED165.A, R319.1
- removed net N$465: LED166.A, R320.1
- removed net N$466: LED167.A, R321.1
- removed net N$467: LED168.A, R322.1
- removed net N$468: IC26.Q5, R313.1
- removed net N$469: IC26.Q1, R308.2
- removed net N$470: IC26.Q2, R309.2
- removed net N$471: IC26.Q3, R310.2
- removed net N$472: IC25.Q4, R299.1
- removed net N$473: IC25.Q6, R301.1
- removed net N$474: IC25.Q7, R302.1
- removed net N$475: IC25.Q1, R305.2
- removed net N$476: IC27.Q5, R324.1
- removed net N$477: IC27.Q3, R327.2
- removed net N$478: IC27.Q2, R328.2
- removed net N$479: IC27.Q0, R330.2
- removed net N$480: IC28.Q0, R331.2
- removed net N$481: IC28.Q7, R335.1
- removed net N$482: IC28.Q6, R336.1
- removed net N$483: IC28.Q4, R338.1
- removed net N$484: LED_STROBE7.Q4, R339.1
- removed net N$485: LED_STROBE7.Q5, R340.1
- removed net N$486: LED_STROBE7.Q6, R341.1
- removed net N$487: LED_STROBE7.Q7, R342.1
- removed net N$488: LED_STROBE7.Q3, R343.2
- removed net N$489: LED_STROBE7.Q2, R344.2
- removed net N$490: LED_STROBE7.Q1, R345.2
- removed net N$491: LED_STROBE7.Q0, R346.2
- removed net N$492: LED169.A, R323.2
- removed net N$493: LED170.A, R324.2
- removed net N$494: LED171.A, R325.2
- removed net N$495: LED172.A, R326.2
- removed net N$496: LED173.A, R327.1
- removed net N$497: LED174.A, R328.1
- removed net N$498: LED175.A, R329.1
- removed net N$499: LED176.A, R330.1
- removed net N$500: LED177.A, R331.1
- removed net N$501: LED178.A, R332.1
- removed net N$502: LED179.A, R333.1
- removed net N$503: LED180.A, R334.1
- removed net N$504: LED181.A, R335.2
- removed net N$505: LED182.A, R336.2
- removed net N$506: LED183.A, R337.2
- removed net N$507: LED184.A, R338.2
- removed net N$508: LED185.A, R339.2
- removed net N$509: LED186.A, R340.2
- removed net N$510: LED187.A, R341.2
- removed net N$511: LED188.A, R342.2
- removed net N$512: LED189.A, R343.1
- removed net N$513: LED190.A, R344.1
- removed net N$514: LED191.A, R345.1
- removed net N$515: LED192.A, R346.1
- removed net N$516: IC28.Q5, R337.1
- removed net N$517: IC28.Q1, R332.2
- removed net N$518: IC28.Q2, R333.2
- removed net N$519: IC28.Q3, R334.2
- removed net N$520: IC27.Q4, R323.1
- removed net N$521: IC27.Q6, R325.1
- removed net N$522: IC27.Q7, R326.1
- removed net N$523: IC27.Q1, R329.2
- removed net N$526: LED173.C, LED174.C, LED175.C, LED176.C, LED177.C, LED178.C, LED179.C, LED180.C, LED189.C, LED190.C, LED191.C, LED192.C
- net +3V3: no longer IC13.OE, IC13.VCC, IC14.OE, IC14.VCC, IC15.OE, IC15.VCC, IC16.OE, IC16.VCC, IC17.OE, IC17.VCC, IC18.OE, IC18.VCC, IC19.OE, IC19.VCC, IC20.OE, IC20.VCC, IC21.OE, IC21.VCC, IC22.OE, IC22.VCC, IC23.OE, IC23.VCC, IC24.OE, IC24.VCC, IC25.OE, IC25.VCC, IC26.OE, IC26.VCC, IC27.OE, IC27.VCC, IC28.OE, IC28.VCC, LED_STROBE.OE, LED_STROBE.VCC, LED_STROBE1.OE, LED_STROBE1.VCC, LED_STROBE2.OE, LED_STROBE2.VCC, LED_STROBE3.OE, LED_STROBE3.VCC, LED_STROBE4.OE, LED_STROBE4.VCC, LED_STROBE5.OE, LED_STROBE5.VCC, LED_STROBE6.OE, LED_STROBE6.VCC, LED_STROBE7.OE, LED_STROBE7.VCC
- net +5V: no longer C155.1, C156.1, C157.1, C158.1, C159.1, C160.1, C161.1, C162.1, C163.1, C164.1, C165.1, C166.1, C167.1, C168.1, C169.1, C170.1, C171.1, C172.1
- net GND: no longer C155.2, C156.2, C157.2, C158.2, C159.2, C160.2, C161.2, C162.2, C163.2, C164.2, C165.2, C166.2, C167.2, C168.2, C169.2, C170.2, C171.2, C172.2, IC13.GND, IC14.GND, IC15.GND, IC16.GND, IC17.GND, IC18.GND, IC19.GND, IC20.GND, IC21.GND, IC22.GND, IC23.GND, IC24.GND, IC25.GND, IC26.GND, IC27.GND, IC28.GND, LED_STROBE.GND, LED_STROBE1.GND, LED_STROBE2.GND, LED_STROBE3.GND, LED_STROBE4.GND, LED_STROBE5.GND, LED_STROBE6.GND, LED_STROBE7.GND
- net LED_CLK: no longer IC13.CP, IC14.CP, IC15.CP, IC16.CP, IC17.CP, IC18.CP, IC19.CP, IC20.CP, IC21.CP, IC22.CP, IC23.CP, IC24.CP, IC25.CP, IC26.CP, IC27.CP, IC28.CP, LED_STROBE.CP, LED_STROBE1.CP, LED_STROBE2.CP, LED_STROBE3.CP, LED_STROBE4.CP, LED_STROBE5.CP, LED_STROBE6.CP, LED_STROBE7.CP
- net LED_DATA1: no longer IC14.DATA, IC16.DATA, IC18.DATA, IC20.DATA, IC22.DATA, IC24.DATA, IC26.DATA, IC28.DATA
- net LED_ROW_1: no longer LED1.C, LED10.C, LED11.C, LED12.C, LED13.C, LED14.C, LED15.C, LED16.C, LED17.C, LED18.C, LED19.C, LED2.C, LED20.C, LED21.C, LED22.C, LED23.C, LED24.C, LED3.C, LED4.C, LED5.C, LED6.C, LED7.C, LED8.C, LED9.C
- net LED_ROW_2: no longer LED25.C, LED26.C, LED27.C, LED28.C, LED29.C, LED30.C, LED31.C, LED32.C, LED33.C, LED34.C, LED35.C, LED36.C, LED37.C, LED38.C, LED39.C, LED40.C, LED41.C, LED42.C, LED43.C, LED44.C, LED45.C, LED46.C, LED47.C, LED48.C
- net LED_ROW_3: no longer LED49.C, LED50.C, LED51.C, LED52.C, LED53.C, LED54.C, LED55.C, LED56.C, LED57.C, LED58.C, LED59.C, LED60.C, LED61.C, LED62.C, LED63.C, LED64.C, LED65.C, LED66.C, LED67.C, LED68.C, LED69.C, LED70.C, LED71.C, LED72.C
- net LED_ROW_4: no longer LED73.C, LED74.C, LED75.C, LED76.C, LED77.C, LED78.C, LED79.C, LED80.C, LED81.C, LED82.C, LED83.C, LED84.C, LED85.C, LED86.C, LED87.C, LED88.C, LED89.C, LED90.C, LED91.C, LED92.C, LED93.C, LED94.C, LED95.C, LED96.C
- net LED_ROW_5: no longer LED100.C, LED101.C, LED102.C, LED103.C, LED104.C, LED105.C, LED106.C, LED107.C, LED108.C, LED109.C, LED110.C, LED111.C, LED112.C, LED113.C, LED114.C, LED115.C, LED116.C, LED117.C, LED118.C, LED119.C, LED120.C, LED97.C, LED98.C, LED99.C
- net LED_ROW_6: no longer LED121.C, LED122.C, LED123.C, LED124.C, LED125.C, LED126.C, LED127.C, LED128.C, LED129.C, LED130.C, LED131.C, LED132.C, LED133.C, LED134.C, LED135.C, LED136.C, LED137.C, LED138.C, LED139.C, LED140.C, LED141.C, LED142.C, LED143.C, LED144.C
- net LED_ROW_7: no longer LED145.C, LED146.C, LED147.C, LED148.C, LED149.C, LED150.C, LED151.C, LED152.C, LED153.C, LED154.C, LED155.C, LED156.C, LED157.C, LED158.C, LED159.C, LED160.C, LED161.C, LED162.C, LED163.C, LED164.C, LED165.C, LED166.C, LED167.C, LED168.C
- net LED_ROW_8: no longer LED169.C, LED170.C, LED171.C, LED172.C, LED181.C, LED182.C, LED183.C, LED184.C, LED185.C, LED186.C, LED187.C, LED188.C
- net LED_STROBE: no longer IC13.STROBE, IC14.STROBE, IC15.STROBE, IC16.STROBE, IC17.STROBE, IC18.STROBE, IC19.STROBE, IC20.STROBE, IC21.STROBE, IC22.STROBE, IC23.STROBE, IC24.STROBE, IC25.STROBE, IC26.STROBE, IC27.STROBE, IC28.STROBE, LED_STROBE.STROBE, LED_STROBE1.STROBE, LED_STROBE2.STROBE, LED_STROBE3.STROBE, LED_STROBE4.STROBE, LED_STROBE5.STROBE, LED_STROBE6.STROBE, LED_STROBE7.STROBE
Other:
- note removed: "LED Drivers"
- note removed: "LED Supply Decoupling"

Commit message: Made progress in re-evaluating the design
Parts:
- removed IC30: 4051D, 40xx:4051D
- removed IC31: 4024D, 40xx:4024D
- removed IC33: 4017D, 40xx:4017D
- removed R366: 10k, rcl:R-EU_R0603
- removed U$22: ULN2803A, audioic:ULN2803A
- added C155, C156: 100n, rcl:C-EUC0603
- added JP1, JP10, JP2, JP3, JP4, JP5, JP6, JP7, JP8, JP9: JUMPER-SMT_2_NC_PASTE_SILK, SparkFun-Jumpers:JUMPER-SMT_2_NC_PASTE_SILK
- added MUX1, MUX2: 4051D, 40xx:4051D
- added MUX1_RIPPLECOUNTER, MUX2_RIPPLECOUNTER: 4024D, 40xx:4024D
- added R154, R155, R160, R161, R163, R164, R165, R166, R167, R168, R169, R170, R171, R172, R173, R174, R29, R53: 33R, rcl:R-EU_R0603
- added U$29: PROTOTYPEAREA, audioic:PROTOTYPEAREA
Connections:
- removed net LED_CLK: R25.2
- removed net LED_DATA1: R26.2
- removed net LED_ROW_1: U$22.OUT1
- removed net LED_ROW_2: U$22.OUT2
- removed net LED_ROW_3: U$22.OUT3
- removed net LED_ROW_4: U$22.OUT4
- removed net LED_ROW_5: U$22.OUT5
- removed net LED_ROW_6: U$22.OUT6
- removed net LED_ROW_7: U$22.OUT7
- removed net LED_ROW_8: U$22.OUT8
- removed net LED_STROBE: IC31A.CLK, IC33A.CLK, R24.2
- removed net N$525: IC33A.Q7, U$22.IN8
- removed net N$527: IC33A.Q5, U$22.IN6
- removed net N$528: IC33A.Q4, U$22.IN5
- removed net N$529: IC33A.Q3, U$22.IN4
- removed net N$530: IC33A.Q2, U$22.IN3
- removed net N$531: IC33A.Q1, U$22.IN2
- removed net N$532: IC33A.Q0, U$22.IN1
- removed net N$548: IC30A.X, U$1G$1.AUXADC0_8
- removed net N$555: IC30A.INH, R58.2
- removed net N$557: IC33A.Q8, IC33A.Q9, IC33A.RES
- removed net N$558: IC30A.A, IC31A.Q1
- removed net N$559: IC30A.B, IC31A.Q2
- removed net N$560: IC30A.C, IC31A.Q3
- removed net N$562: IC33A.Q6, U$22.IN7
- removed net N$563: IC33A.ENA, R366.2
- new net !RST: JP1.2, U$24G$1.!RST, U$29.!RST
- new net MUX1_A: MUX1A.A, MUX1_RIPPLECOUNTERA.Q1, U$29.MUX1_A
- new net MUX1_B: MUX1A.B, MUX1_RIPPLECOUNTERA.Q2, U$29.MUX1_B
- new net MUX1_C: MUX1A.C, MUX1_RIPPLECOUNTERA.Q3, U$29.MUX1_C
- new net MUX1_ENABLE: MUX1A.INH, R58.2, U$29.MUX1_ENABLE
- new net MUX1_X: JP3.2, JP9.1, MUX1A.X, U$29.MUX1_X
- new net MUX2_A_A: MUX2A.A, MUX2_RIPPLECOUNTERA.Q1, U$29.MUX2_A
- new net MUX2_A_B: MUX2A.B, MUX2_RIPPLECOUNTERA.Q2, U$29.MUX2_B
- new net MUX2_A_C: MUX2A.C, MUX2_RIPPLECOUNTERA.Q3, U$29.MUX2_C
- new net MUX2_A_INH: MUX2A.INH, U$29.MUX2_ENABLE
- new net MUX2_A_X: JP10.1, JP8.2, MUX2A.X, U$29.MUX2_X
- new net MUX2_A_X0: MUX2A.X0, U$29.MUX2_X0
- new net MUX2_A_X1: MUX2A.X1, U$29.MUX2_X1
- new net MUX2_A_X2: MUX2A.X2, U$29.MUX2_X2
- new net MUX2_A_X3: MUX2A.X3, U$29.MUX2_X3
- new net MUX2_A_X4: MUX2A.X4, U$29.MUX2_X4
- new net MUX2_A_X5: MUX2A.X5, U$29.MUX2_X5
- new net MUX2_A_X6: MUX2A.X6, U$29.MUX2_X6
- new net MUX2_A_X7: MUX2A.X7, U$29.MUX2_X7
- new net N$123: R29.2, U$29.S_SCL
- new net N$126: R53.2, U$29.S_SDA
- new net N$132: R154.1, U$1G$5.BCLK_OUT3_51
- new net N$134: R155.1, U$1G$5.SDATA_OUT3_52
- new net N$135: MUX2_RIPPLECOUNTERA.Q4, MUX2_RIPPLECOUNTERA.Q5, MUX2_RIPPLECOUNTERA.Q6, MUX2_RIPPLECOUNTERA.Q7, MUX2_RIPPLECOUNTERA.RES
- new net N$136: JP10.2
- new net N$137: JP9.2
- new net N$143: R160.1, U$29.S_MP13
- new net N$144: R161.1, U$29.S_MP12
- new net N$145: R163.1, U$29.S_MP11
- new net N$146: R164.1, U$29.S_MP10
- new net N$147: R165.1, U$29.S_MP9
- new net N$148: R166.1, U$29.S_MP8
- new net N$149: R167.1, U$29.S_MP7
- new net N$150: R168.1, U$29.S_MP6
- new net N$151: R169.1, U$29.S_MP5
- new net N$152: R170.1, U$29.S_MP4
- new net N$153: R171.1, U$29.S_MP3
- new net N$154: R172.1, U$29.S_MP2
- new net N$155: R173.1, U$29.S_MP1
- new net N$156: R174.1, U$29.S_MP0
- new net P_ADC0: U$24G$1.A0, U$29.P_ADC0
- new net P_ADC1: U$24G$1.A1, U$29.P_ADC1
- new net P_ADC2: U$24G$1.A2, U$29.P_ADC2
- new net P_ADC3: U$24G$1.A3, U$29.P_ADC3
- new net P_ADC4: U$24G$1.A4, U$29.P_ADC4
- new net P_ADC5: U$24G$1.A5, U$29.P_ADC5
- new net P_ADC6_DAC: U$24G$1.DAC, U$29.P_ADC6_DAC
- new net P_ADC7_WPK: U$24G$1.WKP, U$29.P_ADC7_WPK
- new net P_D0: U$24G$1.D0, U$29.P_D0
- new net P_D1: U$24G$1.D1, U$29.P_D1
- new net P_D2: U$24G$1.D2, U$29.P_D2
- new net P_D3: U$24G$1.D3, U$29.P_D3
- new net P_D4: U$24G$1.D4, U$29.P_D4
- new net P_D5: U$24G$1.D5, U$29.P_D5
- new net P_D6: U$24G$1.D6, U$29.P_D6
- new net P_D7: U$24G$1.D7, U$29.P_D7
- new net RX: U$24G$1.RX, U$29.RX
- new net SDATA_IN2_BCLK: U$29.SDATA_IN4_BCLK
- new net SDATA_IN2_DATA: U$29.SDATA_IN4_DATA
- new net SDATA_IN2_LRCLK: U$29.SDATA_IN4_LRCLK
- new net SDATA_IN3_BCLK: U$29.SDATA_IN3_BCLK
- new net SDATA_IN3_DATA: U$29.SDATA_IN3_DATA
- new net SDATA_IN3_LRCLK: U$29.SDATA_IN3_LRCLK
- new net SDATA_OUT2_BCLK: R25.2, U$29.SDATA_OUT4_BCLK
- new net SDATA_OUT2_DATA: R26.2, U$29.SDATA_OUT4_DATA
- new net SDATA_OUT2_LRCLK: MUX1_RIPPLECOUNTERA.CLK, MUX2_RIPPLECOUNTERA.CLK, R24.2, U$29.SDATA_OUT4_LRCLK
- new net SDATA_OUT3_BCLK: R154.2, U$29.SDATA_OUT3_BCLK
- new net SDATA_OUT3_DATA: R155.2, U$29.SDATA_OUT3_DATA
- new net SDATA_OUT3_LRCLK: R56.2, U$29.SDATA_OUT3_LRCLK
- new net S_AUX_ADC0: JP3.1, U$1G$1.AUXADC0_8, U$29.S_AUX_ADC0
- new net S_AUX_ADC1: JP4.2, U$1G$1.AUXADC1_9, U$29.S_AUX_ADC1
- new net S_AUX_ADC2: JP5.1, U$1G$1.AUXADC2_10, U$29.S_AUX_ADC2
- new net S_AUX_ADC3: JP6.1, U$1G$1.AUXADC3_11, U$29.S_AUX_ADC3
- new net S_AUX_ADC4: JP7.1, U$1G$1.AUXADC4_12, U$29.S_AUX_ADC4
- new net S_AUX_ADC5: JP8.1, U$1G$1.AUXADC5_13, U$29.S_AUX_ADC5
- new net S_MP0: R174.2
- new net S_MP1: R173.2
- new net S_MP10: R164.2
- new net S_MP11: R163.2
- new net S_MP12: R161.2
- new net S_MP13: R160.2
- new net S_MP2: R172.2
- new net S_MP3: R171.2
- new net S_MP4: R170.2
- new net S_MP5: R169.2
- new net S_MP6: R168.2
- new net S_MP7: R167.2
- new net S_MP8: R166.2
- new net S_MP9: R165.2
- new net S_SCL: R29.1
- new net S_SDA: R53.1
- new net TX: U$24G$1.TX, U$29.TX
- new net VBAT: U$24G$1.VBAT, U$29.VBAT
- new net VIN: JP2.1, U$24G$1.VIN, U$29.VIN
- net +12V: now also U$29.12V
- net +3V3: now also C155.2, MUX1P.VCC, MUX1P.VEE, MUX2P.VCC, U$24G$1.3V3, U$29.3V3D; no longer IC30P.VCC, IC30P.VEE
- net +5V: now also C156.1, JP2.2, MUX1_RIPPLECOUNTERP.VDD, MUX2P.VEE, MUX2_RIPPLECOUNTERP.VDD, U$29.5V; no longer IC31P.VDD, IC33P.VDD, R366.1
- net -12V: now also U$29.-12V
- net 3V3A: now also U$29.3V3A
- net CV0: now also MUX1A.X0, U$29.MUX1_X0; no longer IC30A.X0
- net CV1: now also MUX1A.X1, U$29.MUX1_X1; no longer IC30A.X1
- net CV2: now also MUX1A.X2, U$29.MUX1_X2; no longer IC30A.X2
- net CV3: now also MUX1A.X3, U$29.MUX1_X3; no longer IC30A.X3
- net CV4: now also MUX1A.X4, U$29.MUX1_X4; no longer IC30A.X4
- net CV5: now also MUX1A.X5, U$29.MUX1_X5; no longer IC30A.X5
- net CV6: now also MUX1A.X6, U$29.MUX1_X6; no longer IC30A.X6
- net CV7: now also MUX1A.X7, U$29.MUX1_X7; no longer IC30A.X7
- net ENCODER0_0: now also JP4.1; no longer U$1G$1.AUXADC1_9
- net ENCODER0_1: now also JP5.2; no longer U$1G$1.AUXADC2_10
- net ENCODER1_0: now also JP6.2; no longer U$1G$1.AUXADC3_11
- net ENCODER1_1: now also JP7.2; no longer U$1G$1.AUXADC4_12
- net GND: now also C155.1, C156.2, MUX1P.GND, MUX1_RIPPLECOUNTERP.VSS, MUX2P.GND, MUX2_RIPPLECOUNTERP.VSS, U$24G$1.GND@2, U$24G$1.GND@21, U$29.GND1, U$29.GND2, U$29.GND3, U$29.GND4, U$29.GND5; no longer IC30P.GND, IC31P.VSS, IC33P.VSS, U$22.COM, U$22.GND
- net N$556: now also MUX1_RIPPLECOUNTERA.Q4, MUX1_RIPPLECOUNTERA.Q5, MUX1_RIPPLECOUNTERA.Q6, MUX1_RIPPLECOUNTERA.Q7, MUX1_RIPPLECOUNTERA.RES; no longer IC31A.Q4, IC31A.Q5, IC31A.Q6, IC31A.Q7, IC31A.RES
- net RESET: now also JP1.1
- net SW1: no longer R56.2
