File: DSPBoard.sch (EAGLE design)
At the start: 457 parts, among them IC1 AD1939WBSTZ, IC10 LM833D, IC11 LM833D, IC12 TL074D, IC13 4520D, IC2 24AA1025, IC29 TL074D, IC3 LM4040B10DBZ, IC4 LM833D, IC5 LM833D, IC6 LM833D, IC7 LM833D, IC8 LM833D, IC9 LM833D, U1 LM11173.3NOPB, U2 PEC11R-4315F-N0012, U3 PEC11R-4315F-N0012, X1 2510-, Y1 12.288MHz

Commit message: MAybe I need to rethink this
Parts:
- removed C100, C102, C103, C104, C106, C99: 1nf, rcl:C-EUC0603
- removed C101, C105, C56: 10nF, rcl:C-EUC0603
- removed C107, C108: 100nF, rcl:C-EUC0603
- removed C17, C25: 100nf, rcl:C-EUC0603
- removed C50: 220uF, rcl:CPOL-EUD
- removed C51: 1nF, rcl:C-EUC0603
- removed C52: 470p, rcl:C-EUC0603
- removed C53: 1uF, rcl:C-EUC0603
- removed C54: 100uF, rcl:CPOL-EUD
- removed C55: 100pF, rcl:C-EUC0603
- removed D3, D4, D7, D8: BAV99,215, SamacSys_Parts:BAV99,215
- removed IC10, IC5: LM833D, linear:LM833D
- removed JP10, JP14, JP15, JP16, JP4, JP5, JP6, JP7, JP8, JP9: JUMPER-SMT_2_NC_PASTE_SILK, SparkFun-Jumpers:JUMPER-SMT_2_NC_PASTE_SILK
- removed R103, R114: 100R, rcl:R-EU_R0603
- removed R104, R106, R115, R117, R118, R120, R121, R123, R67: 2.2k, rcl:R-EU_R0603
- removed R105, R116, R119, R122: 68R, rcl:R-EU_R0603
- removed R164, R165, R166, R167, R168, R169, R170, R171, R172, R173, R174, R175, R176, R53: 33R, rcl:R-EU_R0603
- removed R183, R184, R185: 100, rcl:R-EU_R0603
- removed R46: 6k2, rcl:R-EU_R0603
- removed R47, R48: 22R, rcl:R-EU_R0603
- removed R49: 18k, rcl:R-EU_R0603
- removed TP1, TP2, TP3, TP4: TESTPAD_TPSQTP16R, BeagleBone_Blue_R3:TESTPAD_TPSQTP16R
- removed U$14, U$15, U$7: WQP-PJ301M-12_JACK, thonkiconn:WQP-PJ301M-12_JACK
- removed U$24: PHOTON_SMD, Particle-Devices:PHOTON_SMD
- added C133, C180: 1nF, rcl:C-EUC0603
- added C156, C181: 470p, rcl:C-EUC0603
- added C162, C182: 1uF, rcl:C-EUC0603
- added C163, C183: 100uF, rcl:CPOL-EUD
- added C164, C166, C184, C186: 100pF, rcl:C-EUC0603
- added C165, C185, C69: 10nF, rcl:C-EUC0603
- added C177, C178, C58: 100nf, rcl:C-EUC0603
- added C179: 220uF, rcl:CPOL-EUD
- added D10, D13, D14, D9: BAV99,215, SamacSys_Parts:BAV99,215
- added IC14, IC16: LM833D, linear:LM833D
- added LED1, LED2, LED3, LED4, LED5, LED6, LED7, LED8: (no value), led:LEDCHIPLED_0805
- added R186, R208: 18k, rcl:R-EU_R0603
- added R187, R209: 2.7k, rcl:R-EU_R0603
- added R188, R189, R210, R211: 2.2k, rcl:R-EU_R0603
- added R190, R212: 12.7k, rcl:R-EU_R0603
- added R191, R192, R213, R214: 10k, rcl:R-EU_R0603
- added R193, R215: 6k2, rcl:R-EU_R0603
- added R194, R195, R216, R217: 22R, rcl:R-EU_R0603
- added R196, R218: 100, rcl:R-EU_R0603
- added U$22, U$30, U$31: WQP-PJ301M-12_JACK, thonkiconn:WQP-PJ301M-12_JACK
- C132: value 100pF -> 220uF; device rcl:C-EUC0603 -> rcl:CPOL-EUD
- C57, C77: value 100pF -> 100nf
- C59: value 100nf -> 220uF; device rcl:C-EUC0603 -> rcl:CPOL-EUD
- C60: value 100nf -> 1nF
- C61: value 220uF -> 470p; device rcl:CPOL-EUD -> rcl:C-EUC0603
- C62: value 1nF -> 1uF
- C63: value 470p -> 100uF; device rcl:C-EUC0603 -> rcl:CPOL-EUD
- C64: value 1uF -> 100pF
- C65: value 100uF -> 10nF; device rcl:CPOL-EUD -> rcl:C-EUC0603
- C67, C93: value 10nF -> 1nf
- C68: value 100pF -> 1nf
- C70, C71: value 100nf -> 1nf
- C72: value 220uF -> 1nf; device rcl:CPOL-EUD -> rcl:C-EUC0603
- C73: value 1nF -> 10nF
- C74: value 470p -> 1nf
- C75: value 1uF -> 100nF
- C76: value 100uF -> 100nF; device rcl:CPOL-EUD -> rcl:C-EUC0603
- C78: value 10nF -> 100nf
- C79, C80: value 100nF -> 1nf
- C91, C95: value 1nf -> 10nF
- C96: device rcl:C-EUC0805 -> rcl:C-EUC0603
- C97: value 10nF -> 100nF
- C98: value 1nf -> 100nF; device rcl:C-EUC0805 -> rcl:C-EUC0603
- R15: value 18k -> 33R
- R154: value 33R -> 100R
- R155, R159, R160, R163: value 33R -> 2.2k
- R158, R161: value 33R -> 68R
- R25: value 33R -> 10k
- R26, R29: value 33R -> 470
- R30: value 2.7k -> 470
- R32, R42: value 2.2k -> 470
- R43: value 12.7k -> 470
- R44, R45: value 10k -> 470
- R50: value 2.7k -> 18k
- R51: value 2.2k -> 2.7k
- R55, R69: value 12.7k -> 2.2k
- R57: value 10k -> 12.7k
- R62: value 6k2 -> 10k
- R63: value 22R -> 6k2
- R65: value 18k -> 22R
- R66: value 2.7k -> 100
- R68: value 2.2k -> 100R
- R70: value 10k -> 68R
- R71: value 10k -> 2.2k
- R72: value 6k2 -> 2.2k
- R73: value 22R -> 68R
- R74: value 22R -> 2.2k
- U$29: value PROTOTYPEAREA -> WQP-PJ301M-12_JACK; device audioic:PROTOTYPEAREA -> thonkiconn:WQP-PJ301M-12_JACK
- U$5: value WQP-PJ301M-12_JACK -> PHOTON_WITH_HEADERS; device thonkiconn:WQP-PJ301M-12_JACK -> Particle-Devices:PHOTON_WITH_HEADERS
Connections:
- removed net !RST: JP1.2, U$24G$1.!RST, U$29.!RST
- removed net MP12: R156.1, R161.2, U$1G$4.LRCLK_IN2/MP12_66
- removed net MP13: R157.1, R160.2, U$1G$4.LRCLK_IN3/MP13_69
- removed net MP8: JP15.2, R166.2
- removed net MP9: JP16.2, R165.2
- removed net MUX1_X: JP3.2, JP9.1, MUX1A.X, U$29.MUX1_X
- removed net MUX2_A_INH: MUX2A.INH, U$29.MUX2_ENABLE
- removed net MUX2_A_X: JP10.1, JP8.2, MUX2A.X, U$29.MUX2_X
- removed net MUX2_A_X0: MUX2A.X0, U$29.MUX2_X0
- removed net MUX2_A_X1: MUX2A.X1, U$29.MUX2_X1
- removed net MUX2_A_X2: MUX2A.X2, U$29.MUX2_X2
- removed net MUX2_A_X3: MUX2A.X3, U$29.MUX2_X3
- removed net MUX2_A_X4: MUX2A.X4, U$29.MUX2_X4
- removed net MUX2_A_X5: MUX2A.X5, U$29.MUX2_X5
- removed net MUX2_A_X6: MUX2A.X6, U$29.MUX2_X6
- removed net MUX2_A_X7: MUX2A.X7, U$29.MUX2_X7
- removed net N$100: C141.1, IC11B.+IN, R129.2
- removed net N$101: C138.2, R124.2, U$15.2
- removed net N$102: C109.2, R103.2, U$14.2
- removed net N$103: C110.1, IC11A.OUT, R103.1, R104.2
- removed net N$140: R25.1, U$1G$5.BCLK_OUT2_48
- removed net N$143: R160.1, U$29.S_MP13
- removed net N$144: R161.1, U$29.S_MP12
- removed net N$145: R163.1, U$29.S_MP11
- removed net N$146: R164.1, U$29.S_MP10
- removed net N$147: R165.1, U$29.S_MP9
- removed net N$148: R166.1, U$29.S_MP8
- removed net N$149: R167.1, U$29.S_MP7
- removed net N$150: R168.1, U$29.S_MP6
- removed net N$151: R169.1, U$29.S_MP5
- removed net N$152: R170.1, U$29.S_MP4
- removed net N$153: R171.1, U$29.S_MP3
- removed net N$154: R172.1, U$29.S_MP2
- removed net N$155: R173.1, U$29.S_MP1
- removed net N$156: R174.1, U$29.S_MP0
- removed net N$161: R185.2, R46.1
- removed net N$162: R183.2, R62.1
- removed net N$163: R184.2, R72.1
- removed net N$98: C140.2, R128.2, R129.1, R130.2
- removed net N$99: C139.1, IC11B.OUT, R124.1, R125.2
- removed net P_ADC0: U$24G$1.A0, U$29.P_ADC0
- removed net P_ADC1: U$24G$1.A1, U$29.P_ADC1
- removed net P_ADC2: U$24G$1.A2, U$29.P_ADC2
- removed net P_ADC3: U$24G$1.A3, U$29.P_ADC3
- removed net P_ADC4: U$24G$1.A4, U$29.P_ADC4
- removed net P_ADC5: U$24G$1.A5, U$29.P_ADC5
- removed net P_ADC6_DAC: U$24G$1.DAC, U$29.P_ADC6_DAC
- removed net P_ADC7_WPK: U$24G$1.WKP, U$29.P_ADC7_WPK
- removed net P_D0: U$24G$1.D0, U$29.P_D0
- removed net P_D1: U$24G$1.D1, U$29.P_D1
- removed net P_D2: U$24G$1.D2, U$29.P_D2
- removed net P_D3: U$24G$1.D3, U$29.P_D3
- removed net P_D4: U$24G$1.D4, U$29.P_D4
- removed net P_D5: U$24G$1.D5, U$29.P_D5
- removed net P_D6: U$24G$1.D6, U$29.P_D6
- removed net P_D7: U$24G$1.D7, U$29.P_D7
- removed net RX: U$24G$1.RX, U$29.RX
- removed net SDATA_IN2_BCLK: R175.1, U$29.SDATA_IN4_BCLK
- removed net SDATA_IN2_DATA: R176.1, U$29.SDATA_IN4_DATA
- removed net SDATA_IN2_LRCLK: R156.2, U$29.SDATA_IN4_LRCLK
- removed net SDATA_IN3_BCLK: R159.2, U$29.SDATA_IN3_BCLK
- removed net SDATA_IN3_DATA: R158.2, U$29.SDATA_IN3_DATA
- removed net SDATA_IN3_LRCLK: R157.2, U$29.SDATA_IN3_LRCLK
- removed net SDATA_OUT2_BCLK: R25.2, U$29.SDATA_OUT4_BCLK
- removed net SDATA_OUT2_DATA: R26.2, U$29.SDATA_OUT4_DATA
- removed net SDATA_OUT2_LRCLK: IC13A.CLK, IC13B.CLK, R24.2, U$29.SDATA_OUT4_LRCLK
- removed net SDATA_OUT3_BCLK: R154.2, U$29.SDATA_OUT3_BCLK
- removed net SDATA_OUT3_DATA: R155.2, U$29.SDATA_OUT3_DATA
- removed net SDATA_OUT3_LRCLK: R56.2, U$29.SDATA_OUT3_LRCLK
- removed net SEL0: R27.2, R59.2
- removed net S_AUX_ADC0: JP3.1, U$1G$1.AUXADC0_8, U$29.S_AUX_ADC0
- removed net S_AUX_ADC1: JP4.1, U$1G$1.AUXADC1_9, U$29.S_AUX_ADC1
- removed net S_AUX_ADC2: JP5.1, U$1G$1.AUXADC2_10, U$29.S_AUX_ADC2
- removed net S_AUX_ADC3: JP6.1, U$1G$1.AUXADC3_11, U$29.S_AUX_ADC3
- removed net S_AUX_ADC4: JP7.1, U$1G$1.AUXADC4_12, U$29.S_AUX_ADC4
- removed net S_AUX_ADC5: JP8.1, U$1G$1.AUXADC5_13, U$29.S_AUX_ADC5
- removed net TX: U$24G$1.TX, U$29.TX
- removed net VBAT: U$24G$1.VBAT, U$29.VBAT
- new net AUXADC0: MUX1A.X, U$1G$1.AUXADC0_8
- new net AUXADC1: U$1G$1.AUXADC1_9
- new net AUXADC3: U$1G$1.AUXADC3_11
- new net AUXADC4: U$1G$1.AUXADC4_12
- new net AUXADC5: U$1G$1.AUXADC5_13
- new net ENCODER0_2: U$1G$1.AUXADC2_10
- new net LED_DRIVE: MUX2A.X, R27.2
- new net MUX1_ENABLE1: MUX2A.INH, R25.2
- new net MUX_CLK: IC13A.CLK, IC13B.CLK, R15.2
- new net N$168: C133.1, R186.2, R187.1, R193.2
- new net N$169: C156.2, IC14A.+IN, R187.2
- new net N$170: C133.2, IC14A.-IN, IC14A.OUT, R188.2, R195.2
- new net N$171: IC14B.-IN, R188.1, R189.2
- new net N$172: IC14B.OUT, R189.1, R194.2
- new net N$173: C162.2, IC14B.+IN, R190.1
- new net N$174: C162.1, C163.+, R190.2, R191.2, R192.1, R196.1
- new net N$175: C132.-, U$22.2
- new net N$176: C132.+, R186.1
- new net N$177: R193.1, R196.2
- new net N$188: C180.1, R208.2, R209.1, R215.2
- new net N$189: C181.2, IC16A.+IN, R209.2
- new net N$190: C180.2, IC16A.-IN, IC16A.OUT, R210.2, R217.2
- new net N$191: IC16B.-IN, R210.1, R211.2
- new net N$192: IC16B.OUT, R211.1, R216.2
- new net N$193: C182.2, IC16B.+IN, R212.1
- new net N$194: C182.1, C183.+, R212.2, R213.2, R214.1, R218.1
- new net N$195: C179.-, U$31.2
- new net N$196: C179.+, R208.1
- new net N$197: R215.1, R218.2
- net +12V: now also C177.1, C57.1, C76.2, C77.1, C98.2, IC14P.V+, IC16P.V+; no longer C108.2, C17.1, C59.1, C70.1, C80.2, IC10P.V+, IC5P.V+, U$29.12V
- net +3V3: now also R25.1, U$5.3V3; no longer U$24G$1.3V3, U$29.3V3D
- net +5V: no longer U$29.5V
- net -12V: now also C178.2, C58.2, C75.1, C78.2, C97.1, IC14P.V-, IC16P.V-; no longer C107.1, C25.2, C60.2, C71.2, C79.1, IC10P.V-, IC5P.V-, U$29.-12V
- net 3V3A: now also D10.2, D13.1, D14.2, D9.1, R192.2, R214.2, R62.2; no longer D3.1, D4.2, D7.1, D8.2, R45.2, R61.2, R71.2, U$29.3V3A
- net AIN1+: now also C65.2, C66.1, D6.3, R64.1; no longer C56.2, C57.1, D4.3, R47.1
- net AIN1-: now also C64.2, C65.1, D5.3, R65.1; no longer C55.2, C56.1, D3.3, R48.1
- net AIN2+: now also C165.2, C166.1, D10.3, R194.1; no longer C67.2, C68.1, D7.3, R63.1
- net AIN2-: now also C164.2, C165.1, D9.3, R195.1; no longer C66.2, C67.1, D8.3, R64.1
- net AIN3+: now also C185.2, C186.1, D14.3, R216.1; no longer C132.1, C78.2, D6.3, R73.1
- net AIN3-: now also C184.2, C185.1, D13.3, R217.1; no longer C77.2, C78.1, D5.3, R74.1
- net AOUT0+: now also R72.1; no longer R111.1
- net AOUT0-: now also R71.1; no longer R110.1
- net AOUT1+: now also R111.1; no longer R118.1
- net AOUT1-: now also R110.1; no longer R117.1
- net AOUT6+: now also R128.1; no longer R121.1
- net AOUT6-: now also R127.1; no longer R106.1
- net AOUT7+: now also R160.1; no longer R128.1
- net AOUT7-: now also R159.1; no longer R127.1
- net CV0: no longer U$29.MUX1_X0
- net CV1: no longer U$29.MUX1_X1
- net CV2: no longer U$29.MUX1_X2
- net CV3: no longer U$29.MUX1_X3
- net CV4: no longer U$29.MUX1_X4
- net CV5: no longer U$29.MUX1_X5
- net CV6: no longer U$29.MUX1_X6
- net CV7: no longer U$29.MUX1_X7
- net DSP_47: no longer JP15.1
- net DSP_50: no longer JP16.1
- net ENCODER0_0: now also R157.2; no longer JP4.2
- net ENCODER0_1: now also R156.2; no longer JP5.2
- net ENCODER1_0: now also R56.2; no longer JP6.2
- net ENCODER1_1: now also R24.2; no longer JP7.2
- net GND: now also C156.1, C163.-, C164.1, C166.2, C177.2, C178.1, C181.1, C183.-, C184.1, C186.2, C58.1, C61.1, C63.-, C64.1, C66.2, C67.1, C74.2, C75.2, C76.1, C77.2, C78.1, C79.1, C92.2, C93.1, C96.2, C97.2, C98.1, D10.1, D13.2, D14.1, D9.2, R163.1, R191.1, R213.1, R26.1, R29.1, R30.1, R32.1, R42.1, R43.1, R45.1, R61.1, R74.1, U$22.1, U$22.3, U$29.1, U$29.3, U$30.1, U$30.3, U$31.1, U$31.3, U$5.GND@2, U$5.GND@21; no longer C102.2, C103.1, C106.2, C107.2, C108.1, C132.2, C17.2, C25.1, C52.1, C54.-, C55.1, C59.2, C60.1, C63.1, C65.-, C66.1, C68.2, C74.1, C76.-, C77.1, C79.2, C80.1, C91.1, C94.2, C95.1, C98.2, C99.1, D3.2, D4.1, D7.2, D8.1, R120.1, R123.1, R57.1, R70.1, U$14.1, U$14.3, U$15.1, U$15.3, U$24G$1.GND@2, U$24G$1.GND@21, U$29.GND1, U$29.GND2, U$29.GND3, U$29.GND4, U$29.GND5, U$5.1, U$5.3, U$7.1, U$7.3
- net MP0: no longer R174.2
- net MP1: no longer R173.2
- net MP10: no longer R164.2
- net MP11: no longer R163.2
- net MP2: no longer R172.2
- net MP3: no longer R171.2
- net MP4: no longer JP14.1, JP14.2, R170.2
- net MP5: no longer R169.2
- net MP6: no longer R168.2
- net MP7: no longer R167.2
- net MUX1_A: no longer U$29.MUX1_A
- net MUX1_B: no longer U$29.MUX1_B
- net MUX1_C: no longer U$29.MUX1_C
- net MUX1_ENABLE: no longer U$29.MUX1_ENABLE
- net MUX2_A_A: no longer U$29.MUX2_A
- net MUX2_A_B: no longer U$29.MUX2_B
- net MUX2_A_C: no longer U$29.MUX2_C
- net N$104: now also C139.2, IC11B.-IN, R158.2; no longer C110.2, IC11A.-IN, R105.2
- net N$105: now also C140.1, R155.1, R158.1, R159.2; no longer C134.1, R104.1, R105.1, R106.2
- net N$106: now also C140.2, R160.2, R161.1, R163.2; no longer C134.2, R121.2, R122.1, R123.2
- net N$107: now also C139.1, IC11B.OUT, R154.1, R155.2; no longer C135.1, IC11A.+IN, R122.2
- net N$123: now also C141.1, IC11B.+IN, R161.2; no longer R29.2, U$29.S_SCL
- net N$126: now also C138.2, R154.2, U$30.2; no longer R53.2, U$29.S_SDA
- net N$130: now also C109.2, R124.2, U$29.2; no longer R158.1, U$1G$4.SDATA_IN3_70
- net N$132: now also C110.1, IC11A.OUT, R124.1, R125.2; no longer R154.1, U$1G$5.BCLK_OUT3_51
- net N$134: now also C110.2, IC11A.-IN, R126.2; no longer R155.1, U$1G$5.SDATA_OUT3_52
- net N$135: no longer JP20.1, TP4.TP
- net N$136: now also C134.1, R125.1, R126.1, R127.2; no longer JP10.2
- net N$137: now also C134.2, R128.2, R129.1, R130.2; no longer JP9.2
- net N$139: now also C135.1, IC11A.+IN, R129.2; no longer R26.1, U$1G$5.SDATA_OUT2_49
- net N$158: no longer JP19.1, TP3.TP
- net N$159: no longer TP2.TP
- net N$17: now also LED1.A, MUX2A.X0; no longer C100.2, IC10B.-IN, R116.2
- net N$19: now also R156.1, U$1G$4.LRCLK_IN2/MP12_66; no longer C51.1, R15.2, R30.1, R46.2
- net N$20: now also R157.1, U$1G$4.LRCLK_IN3/MP13_69; no longer C52.2, IC5A.+IN, R30.2
- net N$22: now also LED2.A, MUX2A.X1; no longer C101.1, R115.1, R116.1, R117.2
- net N$23: now also JP20.1; no longer C51.2, IC5A.-IN, IC5A.OUT, R32.2, R48.2
- net N$25: now also JP19.1; no longer IC5B.-IN, R32.1, R42.2
- net N$26: now also LED3.A, MUX2A.X2; no longer IC5B.OUT, R42.1, R47.2
- net N$30: now also LED4.A, MUX2A.X3; no longer R175.2, U$1G$4.BCLK_IN2_65
- net N$33: now also LED5.A, MUX2A.X4; no longer R159.1, U$1G$4.BCLK_IN3_68
- net N$34: now also LED6.A, MUX2A.X5; no longer C53.2, IC5B.+IN, R43.1
- net N$36: now also LED7.A, MUX2A.X6; no longer C53.1, C54.+, R185.1, R43.2, R44.2, R45.1
- net N$38: now also LED8.A, MUX2A.X7; no longer C50.-, U$5.2
- net N$39: now also LED1.C, R45.2; no longer R176.2, U$1G$4.SDATA_IN2_67
- net N$40: now also LED2.C, R44.2; no longer C50.+, R15.1
- net N$41: now also LED3.C, R43.2; no longer C62.1, R49.2, R50.1, R62.2
- net N$42: now also C60.1, R51.1, R63.2; no longer C63.2, IC6A.+IN
- net N$43: now also C61.2, IC6A.+IN; no longer C62.2, IC6A.-IN, IC6A.OUT, R64.2
- net N$44: now also C60.2, IC6A.-IN, IC6A.OUT, R65.2; no longer IC6B.-IN, R51.1
- net N$45: now also IC6B.-IN, R55.2; no longer IC6B.OUT, R63.2
- net N$46: now also IC6B.OUT, R64.2; no longer C64.2, IC6B.+IN
- net N$47: now also C62.2, IC6B.+IN, R57.1; no longer C64.1, C65.+, R183.1, R55.2, R57.2, R61.1
- net N$48: now also C62.1, C63.+, R57.2, R61.2, R62.1, R66.1; no longer C61.-, U$6.2
- net N$49: now also C59.-, U$6.2; no longer C61.+, R49.1
- net N$50: now also C59.+, R50.1; no longer C73.1, R65.2, R66.1, R72.2
- net N$51: now also R63.1; no longer C74.2, IC7A.+IN
- net N$52: now also LED4.C, R42.2; no longer C73.2, IC7A.-IN, IC7A.OUT, R67.2, R74.2
- net N$53: now also C72.2, R109.2; no longer R67.1, R68.2
- net N$54: now also C73.1, R108.1, R109.1, R110.2; no longer IC7B.OUT, R68.1, R73.2
- net N$55: now also C73.2, R111.2, R112.1, R113.2; no longer C75.2, IC7B.+IN, R69.1
- net N$56: now also C72.1, IC7B.OUT, R107.1, R108.2; no longer C75.1, C76.+, R184.1, R69.2, R70.2, R71.1
- net N$57: now also C74.1, IC7B.+IN, R112.2; no longer C72.-, U$7.2
- net N$58: now also C71.2, R107.2, U$17.2; no longer C72.+, R65.1
- net N$59: now also C67.2, R68.2, U$16.2; no longer C101.2, R118.2, R119.1, R120.2
- net N$60: now also C68.1, IC7A.OUT, R68.1, R69.2; no longer C100.1, IC10B.OUT, R114.1, R115.2
- net N$61: now also C68.2, IC7A.-IN, R70.2; no longer C102.1, IC10B.+IN, R119.2
- net N$62: now also C69.1, R69.1, R70.1, R71.2; no longer C99.2, R114.2, U$17.2
- net N$63: now also C69.2, R72.2, R73.1, R74.2; no longer C95.2, R107.2, U$16.2
- net N$64: now also C70.1, IC7A.+IN, R73.2; no longer C96.1, IC10A.OUT, R107.1, R108.2
- net N$65: now also C94.2, IC9B.-IN, R98.2; no longer C96.2, IC10A.-IN, R109.2
- net N$66: now also C95.1, R97.1, R98.1, R99.2; no longer C97.1, R108.1, R109.1, R110.2
- net N$67: now also C95.2, R100.2, R101.1, R102.2; no longer C97.2, R111.2, R112.1, R113.2
- net N$68: now also C94.1, IC9B.OUT, R96.1, R97.2; no longer C98.1, IC10A.+IN, R112.2
- net N$7: no longer TP1.TP
- net N$84: now also C96.1, IC9B.+IN, R101.2; no longer C104.2, IC9B.-IN, R98.2
- net N$85: now also C93.2, R96.2, U$13.2; no longer C105.1, R97.1, R98.1, R99.2
- net N$86: now also C79.2, R89.2, U$12.2; no longer C105.2, R100.2, R101.1, R102.2
- net N$87: now also C80.1, IC9A.OUT, R89.1, R90.2; no longer C104.1, IC9B.OUT, R96.1, R97.2
- net N$88: now also C80.2, IC9A.-IN, R91.2; no longer C106.1, IC9B.+IN, R101.2
- net N$89: now also C91.1, R90.1, R91.1, R92.2; no longer C103.2, R96.2, U$13.2
- net N$90: now also R93.2, R94.1, R95.2; no longer R89.2, U$12.2
- net N$91: now also IC9A.+IN, R94.2; no longer IC9A.OUT, R89.1, R90.2
- net N$92: now also LED5.C, R32.2; no longer C92.2, IC9A.-IN, R91.2
- net N$93: now also LED6.C, R30.2; no longer C93.1, R90.1, R91.1, R92.2
- net N$94: now also LED7.C, R29.2; no longer C93.2, R93.2, R94.1, R95.2
- net N$95: now also LED8.C, R26.2; no longer C94.1, IC9A.+IN, R94.2
- net N$96: now also JP1.1, U$5.D1; no longer C139.2, IC11B.-IN, R126.2
- net N$97: now also JP3.1, U$5.D0; no longer C140.1, R125.1, R126.1, R127.2
- net RESET: now also U$5.!RST; no longer JP1.1
- net SW0: now also R59.2
- net S_SCL: now also JP1.2; no longer R29.1
- net S_SDA: now also JP3.2; no longer R53.1
- net VIN: now also U$5.VIN; no longer U$24G$1.VIN, U$29.VIN
Other:
- note removed: "DSP Power Supply Decoupling"
