File: DSPBoard.brd (EAGLE design)
At the start: 220 x 106.1 mm, 824 parts, among them IC1 AD1939WBSTZ, IC10 LM833D, IC11 LM833D, IC12 TL074D, IC13 CD74HC4094M96, IC14 CD74HC4094M96, IC15 CD74HC4094M96, IC16 CD74HC4094M96, IC17 CD74HC4094M96, IC18 CD74HC4094M96, IC19 CD74HC4094M96, IC2 24AA1025, IC20 CD74HC4094M96, IC21 CD74HC4094M96, IC22 CD74HC4094M96, IC23 CD74HC4094M96, IC24 CD74HC4094M96, IC25 CD74HC4094M96, IC26 CD74HC4094M96, IC27 CD74HC4094M96, IC28 CD74HC4094M96, IC29 TL074D, IC3 LM4040B10DBZ, IC30 4051D, IC31 4024D, IC33 4017D, IC4 LM833D, IC5 LM833D, IC6 LM833D, IC7 LM833D, IC8 LM833D, IC9 LM833D, U1 LM11173.3NOPB, U2 PEC11R-4315F-N0012, U3 PEC11R-4315F-N0012, X1 2510-, Y1 12.288MHz

Commit message: removed LEDS
Parts:
- removed C155, C156, C157, C158, C159, C160, C161, C162, C163, C164, C165, C166, C167, C168, C169, C170, C171, C172: 100nf, rcl:C0603
- removed IC13, IC14, IC15, IC16, IC17, IC18, IC19, IC20, IC21, IC22, IC23, IC24, IC25, IC26, IC27, IC28, LED_STROBE, LED_STROBE1, LED_STROBE2, LED_STROBE3, LED_STROBE4, LED_STROBE5, LED_STROBE6, LED_STROBE7: CD74HC4094M96, CD74HC4094M96:SOIC127P600X175-16N
- removed LED1, LED10, LED100, LED101, LED102, LED103, LED104, LED105, LED106, LED107, LED108, LED109, LED11, LED110, LED111, LED112, LED113, LED114, LED115, LED116, LED117, LED118, LED119, LED12, LED120, LED121, LED122, LED123, LED124, LED125, LED126, LED127, LED128, LED129, LED13, LED130, LED131, LED132, LED133, LED134, LED135, LED136, LED137, LED138, LED139, LED14, LED140, LED141, LED142, LED143, LED144, LED145, LED146, LED147, LED148, LED149, LED15, LED150, LED151, LED152, LED153, LED154, LED155, LED156, LED157, LED158, LED159, LED16, LED160, LED161, LED162, LED163, LED164, LED165, LED166, LED167, LED168, LED169, LED17, LED170, LED171, LED172, LED173, LED174, LED175, LED176, LED177, LED178, LED179, LED18, LED180, LED181, LED182, LED183, LED184, LED185, LED186, LED187, LED188, LED189, LED19, LED190, LED191, LED192, LED2, LED20, LED21, LED22, LED23, LED24, LED25, LED26, LED27, LED28, LED29, LED3, LED30, LED31, LED32, LED33, LED34, LED35, LED36, LED37, LED38, LED39, LED4, LED40, LED41, LED42, LED43, LED44, LED45, LED46, LED47, LED48, LED49, LED5, LED50, LED51, LED52, LED53, LED54, LED55, LED56, LED57, LED58, LED59, LED6, LED60, LED61, LED62, LED63, LED64, LED65, LED66, LED67, LED68, LED69, LED7, LED70, LED71, LED72, LED73, LED74, LED75, LED76, LED77, LED78, LED79, LED8, LED80, LED81, LED82, LED83, LED84, LED85, LED86, LED87, LED88, LED89, LED9, LED90, LED91, LED92, LED93, LED94, LED95, LED96, LED97, LED98, LED99: (no value), led:CHIPLED_0805
- removed R154, R155, R156, R157, R158, R159, R160, R161, R163, R164, R165, R166, R167, R168, R169, R170, R171, R172, R173, R174, R175, R176, R181, R182, R183, R184, R185, R186, R187, R188, R189, R190, R195, R196, R197, R198, R199, R200, R201, R202, R203, R204, R205, R206, R207, R208, R209, R210, R211, R212, R213, R214, R219, R220, R221, R222, R223, R224, R225, R226, R227, R228, R229, R230, R231, R232, R233, R234, R235, R236, R237, R238, R243, R244, R245, R246, R247, R248, R249, R250, R251, R252, R253, R254, R255, R256, R257, R258, R259, R260, R261, R262, R267, R268, R269, R270, R271, R272, R273, R274, R275, R276, R277, R278, R279, R280, R281, R282, R283, R284, R285, R286, R291, R292, R293, R294, R295, R296, R297, R298, R299, R300, R301, R302, R303, R304, R305, R306, R307, R308, R309, R310, R315, R316, R317, R318, R319, R320, R321, R322, R323, R324, R325, R326, R327, R328, R329, R330, R331, R332, R333, R334, R339, R340, R341, R342, R343, R344, R345, R346: 470R, rcl:R0603
- removed R177, R178, R179, R180, R191, R192, R193, R194, R215, R216, R217, R218, R239, R240, R241, R242, R263, R264, R265, R266, R287, R288, R289, R290, R311, R312, R313, R314, R335, R336, R337, R338: 470, rcl:R0603
- added U$24: PHOTON_SMD, Particle-Devices:PHOTON_SMD
Connections:
- removed net LED_S1: IC13.2, IC14.9, IC15.2, IC16.9, IC17.2, IC18.9, IC19.2, IC20.9, IC21.2, IC22.9, IC23.2, IC24.9, IC25.2, IC26.9, IC27.2, IC28.9
- removed net LED_S2: IC13.9, IC15.9, IC17.9, IC19.9, IC21.9, IC23.9, IC25.9, IC27.9, LED_STROBE.2, LED_STROBE1.2, LED_STROBE2.2, LED_STROBE3.2, LED_STROBE4.2, LED_STROBE5.2, LED_STROBE6.2, LED_STROBE7.2
- removed net N$123: IC14.13, R179.1
- removed net N$126: IC14.5, R174.2
- removed net N$132: IC14.6, R175.2
- removed net N$134: IC14.7, R176.2
- removed net N$135: IC13.14, R165.1
- removed net N$137: IC13.12, R167.1
- removed net N$142: IC13.11, R168.1
- removed net N$143: IC13.5, R171.2
- removed net N$144: IC15.13, R155.1
- removed net N$145: IC15.7, R158.2
- removed net N$146: IC15.6, R159.2
- removed net N$147: IC15.4, R161.2
- removed net N$148: IC16.4, R163.2
- removed net N$149: IC16.11, R191.1
- removed net N$150: IC16.12, R192.1
- removed net N$151: IC16.14, R194.1
- removed net N$152: LED_STROBE1.14, R195.1
- removed net N$153: LED_STROBE1.13, R196.1
- removed net N$154: LED_STROBE1.12, R197.1
- removed net N$155: LED_STROBE1.11, R198.1
- removed net N$156: LED_STROBE1.7, R199.2
- removed net N$157: LED_STROBE1.6, R200.2
- removed net N$158: LED_STROBE1.5, R201.2
- removed net N$159: LED_STROBE1.4, R202.2
- removed net N$160: LED25.A, R154.2
- removed net N$161: LED26.A, R155.2
- removed net N$163: LED27.A, R156.2
- removed net N$164: LED28.A, R157.2
- removed net N$165: IC13.13, R166.1
- removed net N$166: LED29.A, R158.1
- removed net N$167: LED30.A, R159.1
- removed net N$168: IC13.7, R169.2
- removed net N$169: IC13.6, R170.2
- removed net N$170: LED31.A, R160.1
- removed net N$171: IC13.4, R172.2
- removed net N$172: IC14.4, R173.2
- removed net N$173: LED32.A, R161.1
- removed net N$174: LED33.A, R163.1
- removed net N$175: LED34.A, R164.1
- removed net N$176: IC14.11, R177.1
- removed net N$177: IC14.12, R178.1
- removed net N$178: LED35.A, R189.1
- removed net N$179: IC14.14, R180.1
- removed net N$180: LED_STROBE.14, R181.1
- removed net N$181: LED_STROBE.13, R182.1
- removed net N$182: LED_STROBE.12, R183.1
- removed net N$183: LED_STROBE.11, R184.1
- removed net N$184: LED_STROBE.7, R185.2
- removed net N$185: LED_STROBE.6, R186.2
- removed net N$186: LED_STROBE.5, R187.2
- removed net N$187: LED_STROBE.4, R188.2
- removed net N$188: LED1.A, R165.2
- removed net N$189: LED2.A, R166.2
- removed net N$190: LED3.A, R167.2
- removed net N$191: LED4.A, R168.2
- removed net N$192: LED5.A, R169.1
- removed net N$193: LED6.A, R170.1
- removed net N$194: LED7.A, R171.1
- removed net N$195: LED8.A, R172.1
- removed net N$196: LED9.A, R173.1
- removed net N$197: LED10.A, R174.1
- removed net N$198: LED11.A, R175.1
- removed net N$199: LED12.A, R176.1
- removed net N$200: LED13.A, R177.2
- removed net N$201: LED14.A, R178.2
- removed net N$202: LED15.A, R179.2
- removed net N$203: LED16.A, R180.2
- removed net N$204: LED17.A, R181.2
- removed net N$205: LED18.A, R182.2
- removed net N$206: LED19.A, R183.2
- removed net N$207: LED20.A, R184.2
- removed net N$208: LED21.A, R185.1
- removed net N$209: LED22.A, R186.1
- removed net N$210: LED23.A, R187.1
- removed net N$211: LED24.A, R188.1
- removed net N$213: LED36.A, R190.1
- removed net N$214: LED37.A, R191.2
- removed net N$215: LED38.A, R192.2
- removed net N$216: LED39.A, R193.2
- removed net N$217: LED40.A, R194.2
- removed net N$218: LED41.A, R195.2
- removed net N$219: LED42.A, R196.2
- removed net N$220: LED43.A, R197.2
- removed net N$221: LED44.A, R198.2
- removed net N$222: LED45.A, R199.1
- removed net N$223: LED46.A, R200.1
- removed net N$224: LED47.A, R201.1
- removed net N$225: LED48.A, R202.1
- removed net N$226: IC16.13, R193.1
- removed net N$227: IC16.5, R164.2
- removed net N$228: IC16.6, R189.2
- removed net N$229: IC16.7, R190.2
- removed net N$230: IC15.14, R154.1
- removed net N$231: IC15.12, R156.1
- removed net N$232: IC15.11, R157.1
- removed net N$233: IC15.5, R160.2
- removed net N$236: IC17.13, R204.1
- removed net N$237: IC17.7, R207.2
- removed net N$238: IC17.6, R208.2
- removed net N$239: IC17.4, R210.2
- removed net N$240: IC18.4, R211.2
- removed net N$241: IC18.11, R215.1
- removed net N$242: IC18.12, R216.1
- removed net N$243: IC18.14, R218.1
- removed net N$244: LED_STROBE2.14, R219.1
- removed net N$245: LED_STROBE2.13, R220.1
- removed net N$246: LED_STROBE2.12, R221.1
- removed net N$247: LED_STROBE2.11, R222.1
- removed net N$248: LED_STROBE2.7, R223.2
- removed net N$249: LED_STROBE2.6, R224.2
- removed net N$250: LED_STROBE2.5, R225.2
- removed net N$251: LED_STROBE2.4, R226.2
- removed net N$252: LED49.A, R203.2
- removed net N$253: LED50.A, R204.2
- removed net N$254: LED51.A, R205.2
- removed net N$255: LED52.A, R206.2
- removed net N$256: LED53.A, R207.1
- removed net N$257: LED54.A, R208.1
- removed net N$258: LED55.A, R209.1
- removed net N$259: LED56.A, R210.1
- removed net N$260: LED57.A, R211.1
- removed net N$261: LED58.A, R212.1
- removed net N$262: LED59.A, R213.1
- removed net N$263: LED60.A, R214.1
- removed net N$264: LED61.A, R215.2
- removed net N$265: LED62.A, R216.2
- removed net N$266: LED63.A, R217.2
- removed net N$267: LED64.A, R218.2
- removed net N$268: LED65.A, R219.2
- removed net N$269: LED66.A, R220.2
- removed net N$270: LED67.A, R221.2
- removed net N$271: LED68.A, R222.2
- removed net N$272: LED69.A, R223.1
- removed net N$273: LED70.A, R224.1
- removed net N$274: LED71.A, R225.1
- removed net N$275: LED72.A, R226.1
- removed net N$276: IC18.13, R217.1
- removed net N$277: IC18.5, R212.2
- removed net N$278: IC18.6, R213.2
- removed net N$279: IC18.7, R214.2
- removed net N$280: IC17.14, R203.1
- removed net N$281: IC17.12, R205.1
- removed net N$282: IC17.11, R206.1
- removed net N$283: IC17.5, R209.2
- removed net N$284: IC19.13, R228.1
- removed net N$285: IC19.7, R231.2
- removed net N$286: IC19.6, R232.2
- removed net N$287: IC19.4, R234.2
- removed net N$288: IC20.4, R235.2
- removed net N$289: IC20.11, R239.1
- removed net N$290: IC20.12, R240.1
- removed net N$291: IC20.14, R242.1
- removed net N$292: LED_STROBE3.14, R243.1
- removed net N$293: LED_STROBE3.13, R244.1
- removed net N$294: LED_STROBE3.12, R245.1
- removed net N$295: LED_STROBE3.11, R246.1
- removed net N$296: LED_STROBE3.7, R247.2
- removed net N$297: LED_STROBE3.6, R248.2
- removed net N$298: LED_STROBE3.5, R249.2
- removed net N$299: LED_STROBE3.4, R250.2
- removed net N$300: LED73.A, R227.2
- removed net N$301: LED74.A, R228.2
- removed net N$302: LED75.A, R229.2
- removed net N$303: LED76.A, R230.2
- removed net N$304: LED77.A, R231.1
- removed net N$305: LED78.A, R232.1
- removed net N$306: LED79.A, R233.1
- removed net N$307: LED80.A, R234.1
- removed net N$308: LED81.A, R235.1
- removed net N$309: LED82.A, R236.1
- removed net N$310: LED83.A, R237.1
- removed net N$311: LED84.A, R238.1
- removed net N$312: LED85.A, R239.2
- removed net N$313: LED86.A, R240.2
- removed net N$314: LED87.A, R241.2
- removed net N$315: LED88.A, R242.2
- removed net N$316: LED89.A, R243.2
- removed net N$317: LED90.A, R244.2
- removed net N$318: LED91.A, R245.2
- removed net N$319: LED92.A, R246.2
- removed net N$320: LED93.A, R247.1
- removed net N$321: LED94.A, R248.1
- removed net N$322: LED95.A, R249.1
- removed net N$323: LED96.A, R250.1
- removed net N$324: IC20.13, R241.1
- removed net N$325: IC20.5, R236.2
- removed net N$326: IC20.6, R237.2
- removed net N$327: IC20.7, R238.2
- removed net N$328: IC19.14, R227.1
- removed net N$329: IC19.12, R229.1
- removed net N$330: IC19.11, R230.1
- removed net N$331: IC19.5, R233.2
- removed net N$332: IC21.13, R252.1
- removed net N$333: IC21.7, R255.2
- removed net N$334: IC21.6, R256.2
- removed net N$335: IC21.4, R258.2
- removed net N$336: IC22.4, R259.2
- removed net N$337: IC22.11, R263.1
- removed net N$338: IC22.12, R264.1
- removed net N$339: IC22.14, R266.1
- removed net N$340: LED_STROBE4.14, R267.1
- removed net N$341: LED_STROBE4.13, R268.1
- removed net N$342: LED_STROBE4.12, R269.1
- removed net N$343: LED_STROBE4.11, R270.1
- removed net N$344: LED_STROBE4.7, R271.2
- removed net N$345: LED_STROBE4.6, R272.2
- removed net N$346: LED_STROBE4.5, R273.2
- removed net N$347: LED_STROBE4.4, R274.2
- removed net N$348: LED97.A, R251.2
- removed net N$349: LED98.A, R252.2
- removed net N$350: LED99.A, R253.2
- removed net N$351: LED100.A, R254.2
- removed net N$352: LED101.A, R255.1
- removed net N$353: LED102.A, R256.1
- removed net N$354: LED103.A, R257.1
- removed net N$355: LED104.A, R258.1
- removed net N$356: LED105.A, R259.1
- removed net N$357: LED106.A, R260.1
- removed net N$358: LED107.A, R261.1
- removed net N$359: LED108.A, R262.1
- removed net N$360: LED109.A, R263.2
- removed net N$361: LED110.A, R264.2
- removed net N$362: LED111.A, R265.2
- removed net N$363: LED112.A, R266.2
- removed net N$364: LED113.A, R267.2
- removed net N$365: LED114.A, R268.2
- removed net N$366: LED115.A, R269.2
- removed net N$367: LED116.A, R270.2
- removed net N$368: LED117.A, R271.1
- removed net N$369: LED118.A, R272.1
- removed net N$370: LED119.A, R273.1
- removed net N$371: LED120.A, R274.1
- removed net N$372: IC22.13, R265.1
- removed net N$373: IC22.5, R260.2
- removed net N$374: IC22.6, R261.2
- removed net N$375: IC22.7, R262.2
- removed net N$376: IC21.14, R251.1
- removed net N$377: IC21.12, R253.1
- removed net N$378: IC21.11, R254.1
- removed net N$379: IC21.5, R257.2
- removed net N$380: IC23.13, R276.1
- removed net N$381: IC23.7, R279.2
- removed net N$382: IC23.6, R280.2
- removed net N$383: IC23.4, R282.2
- removed net N$384: IC24.4, R283.2
- removed net N$385: IC24.11, R287.1
- removed net N$386: IC24.12, R288.1
- removed net N$387: IC24.14, R290.1
- removed net N$388: LED_STROBE5.14, R291.1
- removed net N$389: LED_STROBE5.13, R292.1
- removed net N$390: LED_STROBE5.12, R293.1
- removed net N$391: LED_STROBE5.11, R294.1
- removed net N$392: LED_STROBE5.7, R295.2
- removed net N$393: LED_STROBE5.6, R296.2
- removed net N$394: LED_STROBE5.5, R297.2
- removed net N$395: LED_STROBE5.4, R298.2
- removed net N$396: LED121.A, R275.2
- removed net N$397: LED122.A, R276.2
- removed net N$398: LED123.A, R277.2
- removed net N$399: LED124.A, R278.2
- removed net N$400: LED125.A, R279.1
- removed net N$401: LED126.A, R280.1
- removed net N$402: LED127.A, R281.1
- removed net N$403: LED128.A, R282.1
- removed net N$404: LED129.A, R283.1
- removed net N$405: LED130.A, R284.1
- removed net N$406: LED131.A, R285.1
- removed net N$407: LED132.A, R286.1
- removed net N$408: LED133.A, R287.2
- removed net N$409: LED134.A, R288.2
- removed net N$410: LED135.A, R289.2
- removed net N$411: LED136.A, R290.2
- removed net N$412: LED137.A, R291.2
- removed net N$413: LED138.A, R292.2
- removed net N$414: LED139.A, R293.2
- removed net N$415: LED140.A, R294.2
- removed net N$416: LED141.A, R295.1
- removed net N$417: LED142.A, R296.1
- removed net N$418: LED143.A, R297.1
- removed net N$419: LED144.A, R298.1
- removed net N$420: IC24.13, R289.1
- removed net N$421: IC24.5, R284.2
- removed net N$422: IC24.6, R285.2
- removed net N$423: IC24.7, R286.2
- removed net N$424: IC23.14, R275.1
- removed net N$425: IC23.12, R277.1
- removed net N$426: IC23.11, R278.1
- removed net N$427: IC23.5, R281.2
- removed net N$428: IC25.13, R300.1
- removed net N$429: IC25.7, R303.2
- removed net N$430: IC25.6, R304.2
- removed net N$431: IC25.4, R306.2
- removed net N$432: IC26.4, R307.2
- removed net N$433: IC26.11, R311.1
- removed net N$434: IC26.12, R312.1
- removed net N$435: IC26.14, R314.1
- removed net N$436: LED_STROBE6.14, R315.1
- removed net N$437: LED_STROBE6.13, R316.1
- removed net N$438: LED_STROBE6.12, R317.1
- removed net N$439: LED_STROBE6.11, R318.1
- removed net N$440: LED_STROBE6.7, R319.2
- removed net N$441: LED_STROBE6.6, R320.2
- removed net N$442: LED_STROBE6.5, R321.2
- removed net N$443: LED_STROBE6.4, R322.2
- removed net N$444: LED145.A, R299.2
- removed net N$445: LED146.A, R300.2
- removed net N$446: LED147.A, R301.2
- removed net N$447: LED148.A, R302.2
- removed net N$448: LED149.A, R303.1
- removed net N$449: LED150.A, R304.1
- removed net N$450: LED151.A, R305.1
- removed net N$451: LED152.A, R306.1
- removed net N$452: LED153.A, R307.1
- removed net N$453: LED154.A, R308.1
- removed net N$454: LED155.A, R309.1
- removed net N$455: LED156.A, R310.1
- removed net N$456: LED157.A, R311.2
- removed net N$457: LED158.A, R312.2
- removed net N$458: LED159.A, R313.2
- removed net N$459: LED160.A, R314.2
- removed net N$460: LED161.A, R315.2
- removed net N$461: LED162.A, R316.2
- removed net N$462: LED163.A, R317.2
- removed net N$463: LED164.A, R318.2
- removed net N$464: LED165.A, R319.1
- removed net N$465: LED166.A, R320.1
- removed net N$466: LED167.A, R321.1
- removed net N$467: LED168.A, R322.1
- removed net N$468: IC26.13, R313.1
- removed net N$469: IC26.5, R308.2
- removed net N$470: IC26.6, R309.2
- removed net N$471: IC26.7, R310.2
- removed net N$472: IC25.14, R299.1
- removed net N$473: IC25.12, R301.1
- removed net N$474: IC25.11, R302.1
- removed net N$475: IC25.5, R305.2
- removed net N$476: IC27.13, R324.1
- removed net N$477: IC27.7, R327.2
- removed net N$478: IC27.6, R328.2
- removed net N$479: IC27.4, R330.2
- removed net N$480: IC28.4, R331.2
- removed net N$481: IC28.11, R335.1
- removed net N$482: IC28.12, R336.1
- removed net N$483: IC28.14, R338.1
- removed net N$484: LED_STROBE7.14, R339.1
- removed net N$485: LED_STROBE7.13, R340.1
- removed net N$486: LED_STROBE7.12, R341.1
- removed net N$487: LED_STROBE7.11, R342.1
- removed net N$488: LED_STROBE7.7, R343.2
- removed net N$489: LED_STROBE7.6, R344.2
- removed net N$490: LED_STROBE7.5, R345.2
- removed net N$491: LED_STROBE7.4, R346.2
- removed net N$492: LED169.A, R323.2
- removed net N$493: LED170.A, R324.2
- removed net N$494: LED171.A, R325.2
- removed net N$495: LED172.A, R326.2
- removed net N$496: LED173.A, R327.1
- removed net N$497: LED174.A, R328.1
- removed net N$498: LED175.A, R329.1
- removed net N$499: LED176.A, R330.1
- removed net N$500: LED177.A, R331.1
- removed net N$501: LED178.A, R332.1
- removed net N$502: LED179.A, R333.1
- removed net N$503: LED180.A, R334.1
- removed net N$504: LED181.A, R335.2
- removed net N$505: LED182.A, R336.2
- removed net N$506: LED183.A, R337.2
- removed net N$507: LED184.A, R338.2
- removed net N$508: LED185.A, R339.2
- removed net N$509: LED186.A, R340.2
- removed net N$510: LED187.A, R341.2
- removed net N$511: LED188.A, R342.2
- removed net N$512: LED189.A, R343.1
- removed net N$513: LED190.A, R344.1
- removed net N$514: LED191.A, R345.1
- removed net N$515: LED192.A, R346.1
- removed net N$516: IC28.13, R337.1
- removed net N$517: IC28.5, R332.2
- removed net N$518: IC28.6, R333.2
- removed net N$519: IC28.7, R334.2
- removed net N$520: IC27.14, R323.1
- removed net N$521: IC27.12, R325.1
- removed net N$522: IC27.11, R326.1
- removed net N$523: IC27.5, R329.2
- removed net N$526: LED173.C, LED174.C, LED175.C, LED176.C, LED177.C, LED178.C, LED179.C, LED180.C, LED189.C, LED190.C, LED191.C, LED192.C
- new net 3V3: U$24.24
- new net VBAT: U$24.22
- new net VIN: U$24.1
- net +3V3: no longer IC13.15, IC13.16, IC14.15, IC14.16, IC15.15, IC15.16, IC16.15, IC16.16, IC17.15, IC17.16, IC18.15, IC18.16, IC19.15, IC19.16, IC20.15, IC20.16, IC21.15, IC21.16, IC22.15, IC22.16, IC23.15, IC23.16, IC24.15, IC24.16, IC25.15, IC25.16, IC26.15, IC26.16, IC27.15, IC27.16, IC28.15, IC28.16, LED_STROBE.15, LED_STROBE.16, LED_STROBE1.15, LED_STROBE1.16, LED_STROBE2.15, LED_STROBE2.16, LED_STROBE3.15, LED_STROBE3.16, LED_STROBE4.15, LED_STROBE4.16, LED_STROBE5.15, LED_STROBE5.16, LED_STROBE6.15, LED_STROBE6.16, LED_STROBE7.15, LED_STROBE7.16
- net +5V: no longer C155.1, C156.1, C157.1, C158.1, C159.1, C160.1, C161.1, C162.1, C163.1, C164.1, C165.1, C166.1, C167.1, C168.1, C169.1, C170.1, C171.1, C172.1
- net GND: now also U$24.2, U$24.21; no longer C155.2, C156.2, C157.2, C158.2, C159.2, C160.2, C161.2, C162.2, C163.2, C164.2, C165.2, C166.2, C167.2, C168.2, C169.2, C170.2, C171.2, C172.2, IC13.8, IC14.8, IC15.8, IC16.8, IC17.8, IC18.8, IC19.8, IC20.8, IC21.8, IC22.8, IC23.8, IC24.8, IC25.8, IC26.8, IC27.8, IC28.8, LED_STROBE.8, LED_STROBE1.8, LED_STROBE2.8, LED_STROBE3.8, LED_STROBE4.8, LED_STROBE5.8, LED_STROBE6.8, LED_STROBE7.8
- net LED_CLK: no longer IC13.3, IC14.3, IC15.3, IC16.3, IC17.3, IC18.3, IC19.3, IC20.3, IC21.3, IC22.3, IC23.3, IC24.3, IC25.3, IC26.3, IC27.3, IC28.3, LED_STROBE.3, LED_STROBE1.3, LED_STROBE2.3, LED_STROBE3.3, LED_STROBE4.3, LED_STROBE5.3, LED_STROBE6.3, LED_STROBE7.3
- net LED_DATA1: no longer IC14.2, IC16.2, IC18.2, IC20.2, IC22.2, IC24.2, IC26.2, IC28.2
- net LED_ROW_1: no longer LED1.C, LED10.C, LED11.C, LED12.C, LED13.C, LED14.C, LED15.C, LED16.C, LED17.C, LED18.C, LED19.C, LED2.C, LED20.C, LED21.C, LED22.C, LED23.C, LED24.C, LED3.C, LED4.C, LED5.C, LED6.C, LED7.C, LED8.C, LED9.C
- net LED_ROW_2: no longer LED25.C, LED26.C, LED27.C, LED28.C, LED29.C, LED30.C, LED31.C, LED32.C, LED33.C, LED34.C, LED35.C, LED36.C, LED37.C, LED38.C, LED39.C, LED40.C, LED41.C, LED42.C, LED43.C, LED44.C, LED45.C, LED46.C, LED47.C, LED48.C
- net LED_ROW_3: no longer LED49.C, LED50.C, LED51.C, LED52.C, LED53.C, LED54.C, LED55.C, LED56.C, LED57.C, LED58.C, LED59.C, LED60.C, LED61.C, LED62.C, LED63.C, LED64.C, LED65.C, LED66.C, LED67.C, LED68.C, LED69.C, LED70.C, LED71.C, LED72.C
- net LED_ROW_4: no longer LED73.C, LED74.C, LED75.C, LED76.C, LED77.C, LED78.C, LED79.C, LED80.C, LED81.C, LED82.C, LED83.C, LED84.C, LED85.C, LED86.C, LED87.C, LED88.C, LED89.C, LED90.C, LED91.C, LED92.C, LED93.C, LED94.C, LED95.C, LED96.C
- net LED_ROW_5: no longer LED100.C, LED101.C, LED102.C, LED103.C, LED104.C, LED105.C, LED106.C, LED107.C, LED108.C, LED109.C, LED110.C, LED111.C, LED112.C, LED113.C, LED114.C, LED115.C, LED116.C, LED117.C, LED118.C, LED119.C, LED120.C, LED97.C, LED98.C, LED99.C
- net LED_ROW_6: no longer LED121.C, LED122.C, LED123.C, LED124.C, LED125.C, LED126.C, LED127.C, LED128.C, LED129.C, LED130.C, LED131.C, LED132.C, LED133.C, LED134.C, LED135.C, LED136.C, LED137.C, LED138.C, LED139.C, LED140.C, LED141.C, LED142.C, LED143.C, LED144.C
- net LED_ROW_7: no longer LED145.C, LED146.C, LED147.C, LED148.C, LED149.C, LED150.C, LED151.C, LED152.C, LED153.C, LED154.C, LED155.C, LED156.C, LED157.C, LED158.C, LED159.C, LED160.C, LED161.C, LED162.C, LED163.C, LED164.C, LED165.C, LED166.C, LED167.C, LED168.C
- net LED_ROW_8: no longer LED169.C, LED170.C, LED171.C, LED172.C, LED181.C, LED182.C, LED183.C, LED184.C, LED185.C, LED186.C, LED187.C, LED188.C
- net LED_STROBE: no longer IC13.1, IC14.1, IC15.1, IC16.1, IC17.1, IC18.1, IC19.1, IC20.1, IC21.1, IC22.1, IC23.1, IC24.1, IC25.1, IC26.1, IC27.1, IC28.1, LED_STROBE.1, LED_STROBE1.1, LED_STROBE2.1, LED_STROBE3.1, LED_STROBE4.1, LED_STROBE5.1, LED_STROBE6.1, LED_STROBE7.1

Commit message: Made progress in re-evaluating the design
Parts:
- removed IC33: 4017D, 40xx:SO16
- removed R366: 10k, rcl:R0603
- removed U$22: ULN2803A, audioic:SO18W300
- added C155, C156: 100n, rcl:C0603
- added JP1, JP10, JP2, JP3, JP4, JP5, JP6, JP7, JP8, JP9: JUMPER-SMT_2_NC_PASTE_SILK, SparkFun-Jumpers:SMT-JUMPER_2_NC_PASTE_SILK
- added MUX2: 4051D, 40xx:SO16
- added MUX2_RIPPLECOUNTER: 4024D, 40xx:SO14
- added R154, R155, R160, R161, R163, R164, R165, R166, R167, R168, R169, R170, R171, R172, R173, R174, R29, R53: 33R, rcl:R0603
- added U$29: PROTOTYPEAREA, audioic:PROTOTYPEAREA
- moved C44 464.8 mm to (-290.1, -173.8)
- moved X1 285.8 mm to (140.8, 13.1), turned to 180 degrees
- moved C124 230.2 mm to (4.97, 108.5), turned to 270 degrees
- moved R136 227.4 mm to (9.27, 114.7), turned to 270 degrees
- moved C125 226.4 mm to (7.07, 108.5), turned to 270 degrees
- moved U2 226.1 mm to (9.79, 113.6), turned to 0 degrees
- moved R21 224.1 mm to (9.99, 112.0), turned to 0 degrees
- moved R28 223.9 mm to (11.6, 114.7), turned to 270 degrees
- moved R140 222.5 mm to (17.2, 118.7), turned to 90 degrees
- moved R10 219.9 mm to (11.4, 109.9), turned to 180 degrees
- moved U$21 215.1 mm to (205.2, 15.6), turned to 90 degrees
- moved U$7 207.2 mm to (205.2, 27.0), turned to 90 degrees
- moved U$6 201.7 mm to (205.2, 38.4), turned to 90 degrees
- moved U$5 198.6 mm to (205.2, 49.8), turned to 90 degrees
- moved VR1 163.4 mm to (26.3, 39.4), turned to 0 degrees
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- renumbered IC30 to MUX1, IC31 to MUX1_RIPPLECOUNTER
Connections:
- removed net 3V3: U$24.24
- removed net LED_CLK: R25.2
- removed net LED_DATA1: R26.2
- removed net LED_ROW_1: U$22.18
- removed net LED_ROW_2: U$22.17
- removed net LED_ROW_3: U$22.16
- removed net LED_ROW_4: U$22.15
- removed net LED_ROW_5: U$22.14
- removed net LED_ROW_6: U$22.13
- removed net LED_ROW_7: U$22.12
- removed net LED_ROW_8: U$22.11
- removed net LED_STROBE: IC33.14, MUX1_RIPPLECOUNTER.1, R24.2
- removed net N$525: IC33.6, U$22.8
- removed net N$527: IC33.1, U$22.6
- removed net N$528: IC33.10, U$22.5
- removed net N$529: IC33.7, U$22.4
- removed net N$530: IC33.4, U$22.3
- removed net N$531: IC33.2, U$22.2
- removed net N$532: IC33.3, U$22.1
- removed net N$548: MUX1.3, U$1.8
- removed net N$555: MUX1.6, R58.2
- removed net N$557: IC33.11, IC33.15, IC33.9
- removed net N$558: MUX1.11, MUX1_RIPPLECOUNTER.12
- removed net N$559: MUX1.10, MUX1_RIPPLECOUNTER.11
- removed net N$560: MUX1.9, MUX1_RIPPLECOUNTER.9
- removed net N$562: IC33.5, U$22.7
- removed net N$563: IC33.13, R366.2
- new net !RST: JP1.2, U$24.23, U$29.P$29
- new net MUX1_A: MUX1.11, MUX1_RIPPLECOUNTER.12, U$29.USER_PAD1233
- new net MUX1_B: MUX1.10, MUX1_RIPPLECOUNTER.11, U$29.USER_PAD1234
- new net MUX1_C: MUX1.9, MUX1_RIPPLECOUNTER.9, U$29.USER_PAD1235
- new net MUX1_ENABLE: MUX1.6, R58.2, U$29.USER_PAD1236
- new net MUX1_X: JP3.2, JP9.1, MUX1.3, U$29.USER_PAD1237
- new net MUX2_A_A: MUX2.11, MUX2_RIPPLECOUNTER.12, U$29.USER_PAD1246
- new net MUX2_A_B: MUX2.10, MUX2_RIPPLECOUNTER.11, U$29.USER_PAD1247
- new net MUX2_A_C: MUX2.9, MUX2_RIPPLECOUNTER.9, U$29.USER_PAD1248
- new net MUX2_A_INH: MUX2.6, U$29.USER_PAD1249
- new net MUX2_A_X: JP10.1, JP8.2, MUX2.3, U$29.USER_PAD1250
- new net MUX2_A_X0: MUX2.13, U$29.USER_PAD1251
- new net MUX2_A_X1: MUX2.14, U$29.USER_PAD1252
- new net MUX2_A_X2: MUX2.15, U$29.USER_PAD1253
- new net MUX2_A_X3: MUX2.12, U$29.USER_PAD1254
- new net MUX2_A_X4: MUX2.1, U$29.USER_PAD1255
- new net MUX2_A_X5: MUX2.5, U$29.USER_PAD1256
- new net MUX2_A_X6: MUX2.2, U$29.USER_PAD1257
- new net MUX2_A_X7: MUX2.4, U$29.USER_PAD1258
- new net N$123: R29.2, U$29.P$13
- new net N$126: R53.2, U$29.P$14
- new net N$132: R154.1, U$1.51
- new net N$134: R155.1, U$1.52
- new net N$135: MUX2_RIPPLECOUNTER.2, MUX2_RIPPLECOUNTER.3, MUX2_RIPPLECOUNTER.4, MUX2_RIPPLECOUNTER.5, MUX2_RIPPLECOUNTER.6
- new net N$136: JP10.2
- new net N$137: JP9.2
- new net N$143: R160.1, U$29.P$28
- new net N$144: R161.1, U$29.P$27
- new net N$145: R163.1, U$29.P$26
- new net N$146: R164.1, U$29.P$25
- new net N$147: R165.1, U$29.P$24
- new net N$148: R166.1, U$29.P$23
- new net N$149: R167.1, U$29.P$22
- new net N$150: R168.1, U$29.P$21
- new net N$151: R169.1, U$29.P$20
- new net N$152: R170.1, U$29.P$19
- new net N$153: R171.1, U$29.P$18
- new net N$154: R172.1, U$29.P$17
- new net N$155: R173.1, U$29.P$16
- new net N$156: R174.1, U$29.P$15
- new net P_ADC0: U$24.12, U$29.P$36
- new net P_ADC1: U$24.11, U$29.P$37
- new net P_ADC2: U$24.10, U$29.P$38
- new net P_ADC3: U$24.9, U$29.P$39
- new net P_ADC4: U$24.8, U$29.P$40
- new net P_ADC5: U$24.7, U$29.P$41
- new net P_ADC6_DAC: U$24.6, U$29.P$42
- new net P_ADC7_WPK: U$24.5, U$29.P$43
- new net P_D0: U$24.13, U$29.P$3
- new net P_D1: U$24.14, U$29.P$4
- new net P_D2: U$24.15, U$29.P$5
- new net P_D3: U$24.16, U$29.P$6
- new net P_D4: U$24.17, U$29.P$7
- new net P_D5: U$24.18, U$29.P$8
- new net P_D6: U$24.19, U$29.P$9
- new net P_D7: U$24.20, U$29.P$10
- new net RX: U$24.4, U$29.P$12
- new net SDATA_IN2_BCLK: U$29.USER_PAD1291
- new net SDATA_IN2_DATA: U$29.USER_PAD1292
- new net SDATA_IN2_LRCLK: U$29.USER_PAD1293
- new net SDATA_IN3_BCLK: U$29.USER_PAD1288
- new net SDATA_IN3_DATA: U$29.USER_PAD1289
- new net SDATA_IN3_LRCLK: U$29.USER_PAD1290
- new net SDATA_OUT2_BCLK: R25.2, U$29.USER_PAD1297
- new net SDATA_OUT2_DATA: R26.2, U$29.USER_PAD1298
- new net SDATA_OUT2_LRCLK: MUX1_RIPPLECOUNTER.1, MUX2_RIPPLECOUNTER.1, R24.2, U$29.USER_PAD1299
- new net SDATA_OUT3_BCLK: R154.2, U$29.USER_PAD1294
- new net SDATA_OUT3_DATA: R155.2, U$29.USER_PAD1295
- new net SDATA_OUT3_LRCLK: R56.2, U$29.USER_PAD1296
- new net S_AUX_ADC0: JP3.1, U$1.8, U$29.P$44
- new net S_AUX_ADC1: JP4.2, U$1.9, U$29.P$45
- new net S_AUX_ADC2: JP5.1, U$1.10, U$29.P$46
- new net S_AUX_ADC3: JP6.1, U$1.11, U$29.P$47
- new net S_AUX_ADC4: JP7.1, U$1.12, U$29.P$48
- new net S_AUX_ADC5: JP8.1, U$1.13, U$29.P$49
- new net S_MP0: R174.2
- new net S_MP1: R173.2
- new net S_MP10: R164.2
- new net S_MP11: R163.2
- new net S_MP12: R161.2
- new net S_MP13: R160.2
- new net S_MP2: R172.2
- new net S_MP3: R171.2
- new net S_MP4: R170.2
- new net S_MP5: R169.2
- new net S_MP6: R168.2
- new net S_MP7: R167.2
- new net S_MP8: R166.2
- new net S_MP9: R165.2
- new net S_SCL: R29.1
- new net S_SDA: R53.1
- new net TX: U$24.3, U$29.P$11
- net +12V: now also U$29.P$51
- net +3V3: now also C155.2, MUX2.16, U$24.24, U$29.P$56
- net +5V: now also C156.1, JP2.2, MUX2.7, MUX2_RIPPLECOUNTER.14, U$29.P$55; no longer IC33.16, R366.1
- net -12V: now also U$29.P$52
- net 3V3A: now also U$29.P$53
- net CV0: now also U$29.USER_PAD1238
- net CV1: now also U$29.USER_PAD1239
- net CV2: now also U$29.USER_PAD1240
- net CV3: now also U$29.USER_PAD1241
- net CV4: now also U$29.USER_PAD1242
- net CV5: now also U$29.USER_PAD1243
- net CV6: now also U$29.USER_PAD1244
- net CV7: now also U$29.USER_PAD1245
- net ENCODER0_0: now also JP4.1; no longer U$1.9
- net ENCODER0_1: now also JP5.2; no longer U$1.10
- net ENCODER1_0: now also JP6.2; no longer U$1.11
- net ENCODER1_1: now also JP7.2; no longer U$1.12
- net GND: now also C155.1, C156.2, MUX2.8, MUX2_RIPPLECOUNTER.7, U$29.P$35, U$29.P$50, U$29.P$54, U$29.USER_PAD1232, U$29.USER_PAD1287; no longer IC33.8, U$22.10, U$22.9
- net RESET: now also JP1.1
- net SW1: no longer R56.2
- net VBAT: now also U$29.P$2
- net VIN: now also JP2.1, U$29.P$1
Routing:
- net ENCODER0_1: track 51.3 -> 0.18 mm, vias 1 -> 0
- net ENCODER0_0: track 49.4 -> 0.00 mm, vias 1 -> 0
- net ENCODER1_0: track 34.5 -> 0.00 mm, vias 1 -> 0
- net ENCODER1_1: track 33.6 -> 0.00 mm, vias 1 -> 0
- net N$547: track 28.9 -> 0.00 mm, vias 1 -> 0
- net N$550: track 28.6 -> 0.00 mm, vias 1 -> 0
- net GND: track 24.3 -> 0.26 mm, vias 1 -> 0
- net N$27: track 10.7 -> 0.00 mm, vias 1 -> 0
- net N$133: track 9.28 -> 0.01 mm
- net N$69: track 8.09 -> 0.20 mm
- net N$28: track 5.67 -> 0.70 mm, vias 1 -> 0
- net N$29: track 4.19 -> 0.35 mm
- net +3V3: track 3.39 -> 0.11 mm
- net SW0: track 1.86 -> 0.00 mm
- net N$552: track 1.55 -> 0.00 mm
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Other:
- board size 220 x 106.1 mm -> 213 x 128.5 mm

Commit message: started laying out the psu
Parts:
- moved MUX2_RIPPLECOUNTER 399.5 mm to (56.2, 40.6)
- moved J1 380.1 mm to (112.4, 20.2)
- moved U1 339.2 mm to (137.4, 19.2), flipped to the bottom, turned to 180 degrees
- moved MUX2 338.1 mm to (56.4, 49.8)
- moved C30 334.7 mm to (120.8, 7.32), turned to 90 degrees
- moved IC4 330.8 mm to (109.9, -19.9), flipped to the bottom
- moved C31 317.8 mm to (123.8, 11.4), turned to 180 degrees
- moved C29 309.5 mm to (128.5, 11.7)
- moved C137 308.3 mm to (138.3, 24.1), turned to 180 degrees
- moved C26 305.4 mm to (112.1, 9.63), turned to 90 degrees
- moved R5 303.5 mm to (127.2, 6.32)
- moved SV1 300.1 mm to (115.8, 12.8), turned to 90 degrees
- moved C32 299.6 mm to (134.0, 24.3)
- moved U$11 295.4 mm to (124.6, 19.1), turned to 90 degrees
- moved C27 287.4 mm to (101.7, 10.3), turned to 270 degrees
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Connections:
- net GND: now also SV1.3, SV1.4, SV1.7, SV1.8
Routing:
- net +5V: track 0.00 -> 33.0 mm, vias 0 -> 2
- net +12V: track 0.00 -> 31.2 mm, vias 0 -> 2
- net N$5: track 0.00 -> 13.7 mm, vias 0 -> 1
- net GND: track 0.26 -> 11.0 mm, vias 0 -> 1
- net N$4: track 0.00 -> 10.3 mm, vias 0 -> 2
- net -10V: track 0.00 -> 7.20 mm, vias 0 -> 1
- net +3V3: track 0.11 -> 7.30 mm
- net 3V3A: track 0.00 -> 5.11 mm, vias 0 -> 1
- net -12V: track 0.00 -> 5.11 mm
- net N$8: track 0.00 -> 4.24 mm, vias 0 -> 1
- net N$6: track 0.00 -> 4.16 mm, vias 0 -> 1
- net N$2: track 0.00 -> 4.12 mm, vias 0 -> 1
- net N$3: track 0.00 -> 1.41 mm

Commit message: some layout changes, need to make daves recomended changes
Parts:
- removed R363: 2.2k, rcl:R0603
- added C157, C158: 100nF, rcl:C0603
- added C159: 0.1u, rcl:C0603
- added JP11, JP12, JP13, JP14, JP15, JP16: JUMPER-SMT_2_NC_PASTE_SILK, SparkFun-Jumpers:SMT-JUMPER_2_NC_PASTE_SILK
- added R156, R157, R158, R159, R175, R176, R180: 33R, rcl:R0603
- added R177: 240R, rcl:R0603
- added R178: 100R, rcl:R0603
- added R179: 75R, rcl:R0603
- added R181: 10k, rcl:R0603
- added SPDIF: (no value), con-lstb:MA04-1
- R13: value 33R -> 10k
- moved R1 420.8 mm to (167.5, 29.1), flipped to the bottom, turned to 270 degrees
- moved C7 400.2 mm to (154.1, 40.8), turned to 270 degrees
- moved R23 377.1 mm to (180.3, 33.7), flipped to the bottom
- moved C22 371.1 mm to (167.9, 48.8), turned to 90 degrees
- moved R20 370.0 mm to (178.4, 35.8), flipped to the bottom
- moved C21 365.4 mm to (162.2, 37.1)
- moved R19 363.5 mm to (177.2, 37.9), flipped to the bottom
- moved R18 357.6 mm to (176.7, 40.0), flipped to the bottom
- moved C16 350.1 mm to (170.0, 48.8), turned to 90 degrees
- moved C19 348.7 mm to (156.4, 37.9)
- moved C20 348.3 mm to (156.7, 51.4), turned to 180 degrees
- moved C14 346.8 mm to (167.9, 39.5), turned to 270 degrees
- moved C11 333.0 mm to (165.9, 53.3)
- moved C18 325.7 mm to (165.3, 37.6)
- moved R142 324.8 mm to (148.5, 47.3), flipped to the bottom, turned to 180 degrees
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Connections:
- removed net N$135: MUX2_RIPPLECOUNTER.2, MUX2_RIPPLECOUNTER.3, MUX2_RIPPLECOUNTER.4, MUX2_RIPPLECOUNTER.5, MUX2_RIPPLECOUNTER.6
- removed net N$162: R162.1, U$1.46
- removed net N$546: R13.2, U$1.23
- removed net N$547: R364.1, U$1.28
- removed net N$550: R368.1, U$1.29
- removed net N$551: R60.2, U$1.45
- removed net N$556: MUX1_RIPPLECOUNTER.2, MUX1_RIPPLECOUNTER.3, MUX1_RIPPLECOUNTER.4, MUX1_RIPPLECOUNTER.5, MUX1_RIPPLECOUNTER.6
- removed net N$7: IC2.8, R363.1
- removed net S_MP0: R174.2
- removed net S_MP1: R173.2
- removed net S_MP10: R164.2
- removed net S_MP11: R163.2
- removed net S_MP12: R161.2
- removed net S_MP13: R160.2
- removed net S_MP2: R172.2
- removed net S_MP3: R171.2
- removed net S_MP4: R170.2
- removed net S_MP5: R169.2
- removed net S_MP6: R168.2
- removed net S_MP7: R167.2
- removed net S_MP8: R166.2
- removed net S_MP9: R165.2
- new net DSP_47: JP15.1, R24.1, U$1.47
- new net DSP_50: JP16.1, R56.1, U$1.50
- new net MP0: R17.1, R174.2, U$1.26
- new net MP1: R173.2, R59.1, U$1.27
- new net MP10: R164.2, R8.2, U$1.58
- new net MP11: R163.2, R27.1, U$1.61
- new net MP12: R156.1, R161.2, U$1.66
- new net MP13: R157.1, R160.2, U$1.69
- new net MP2: R172.2, R364.1, U$1.28
- new net MP3: R171.2, R368.1, U$1.29
- new net MP4: JP14.1, JP14.2, R170.2, R18.2, U$1.39
- new net MP5: R142.2, R169.2, U$1.42
- new net MP6: R168.2, R60.2, U$1.45
- new net MP7: R162.1, R167.2, U$1.46
- new net MP8: JP15.2, R166.2
- new net MP9: JP16.2, R165.2
- new net N$142: JP12.2, R13.2, U$1.33
- new net N$157: JP13.2, R181.2, U$1.32
- net +3V3: now also C159.2, IC2.8, R13.1, R181.1; no longer R363.2
- net 1452_CLK_OUT: now also R180.2; no longer R13.1
- net GND: now also C159.1, JP11.1, JP12.1, JP13.1, R178.1, R179.2, SPDIF.2, SPDIF.3; no longer U$1.32, U$1.33
- net N$129: now also C158.2, R177.2; no longer R18.2, U$1.39
- net N$130: now also R158.1, U$1.70; no longer R142.2, U$1.42
- net N$138: now also R177.1, R178.2, SPDIF.1; no longer R27.1, U$1.61
- net N$141: now also R180.1, U$1.23; no longer R24.1, U$1.47
- net N$30: now also R175.2, U$1.65; no longer R17.1, U$1.26
- net N$31: now also C157.1, U$1.4; no longer R59.1, U$1.27
- net N$32: now also C158.1, U$1.5; no longer R370.2, X1.1
- net N$33: now also R159.1, U$1.68; no longer R8.2, U$1.58
- net N$37: now also C157.2, R179.1, SPDIF.4; no longer R369.2, X1.3
- net N$39: now also R176.2, U$1.67; no longer R56.1, U$1.50
- net N$545: now also JP11.2
- net SDATA_IN2_BCLK: now also R175.1
- net SDATA_IN2_DATA: now also R176.1
- net SDATA_IN2_LRCLK: now also R156.2
- net SDATA_IN3_BCLK: now also R159.2
- net SDATA_IN3_DATA: now also R158.2
- net SDATA_IN3_LRCLK: now also R157.2
- net SEL1: now also MUX1_RIPPLECOUNTER.2
- net SEL2: now also MUX2_RIPPLECOUNTER.2
- net S_SCL: now also R370.2, X1.1
- net S_SDA: now also R369.2, X1.3
Routing:
- net GND: track 11.0 -> 153.9 mm, vias 1 -> 13
- net +3V3: track 7.30 -> 117.9 mm, vias 0 -> 10
- net N$212: track 0.00 -> 52.7 mm, vias 0 -> 5
- net N$32: track 0.00 -> 45.6 mm, vias 0 -> 1
- net N$31: track 0.00 -> 38.6 mm, vias 0 -> 1
- net +12V: track 31.2 -> 50.8 mm
- net 3V3A: track 5.11 -> 18.7 mm, vias 1 -> 2
- net +5V: track 33.0 -> 41.3 mm, vias 2 -> 3
- net DLRCLK: track 0.00 -> 7.90 mm
- net DBCLK: track 0.00 -> 6.76 mm
- net N$1: track 0.00 -> 5.66 mm
- net DSDATA1: track 0.00 -> 4.92 mm
- net N$37: track 0.00 -> 4.92 mm
- net N$138: track 0.00 -> 4.72 mm
- net N$27: track 0.00 -> 3.34 mm
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Other:
- board size 213 x 128.5 mm -> 416 x 128.5 mm
- board text added: "Power Supplies"
