File: DSPBoard.brd (EAGLE design)
At the start: 213.4 x 110 mm, 436 parts, among them IC1 AD1939WBSTZ, IC11 LM833D, IC12 TL074D, IC13 4520D, IC14 LM833D, IC16 LM833D, IC2 24AA1025, IC29 TL074D, IC3 LM4040B10DBZ, IC4 LM833D, IC6 LM833D, IC7 LM833D, IC8 LM833D, IC9 LM833D, U1 LM11173.3NOPB, U2 PEC11R-4315F-N0012, U3 PEC11R-4315F-N0012, X1 2510-, Y1 12.288MHz

Commit message: bom
Parts:
- moved C119 207.4 mm to (106.5, 63.2), turned to 225 degrees
- moved X1 187.1 mm to (71.9, 7.90), turned to 180 degrees
- moved C137 85.6 mm to (21.4, 4.37)
- moved C27 85.6 mm to (15.1, 46.9)
- moved C28 85.6 mm to (18.7, 41.0)
- moved C29 85.6 mm to (19.9, 18.4)
- moved C30 85.6 mm to (16.0, 22.9)
- moved C31 85.6 mm to (19.5, 25.4)
- moved C32 85.6 mm to (25.7, 10.4)
- moved R2 85.6 mm to (13.8, 49.0)
- moved R3 85.6 mm to (16.8, 49.0)
- moved R4 85.6 mm to (20.9, 16.2)
- moved R5 85.6 mm to (19.0, 15.8)
- moved SV1 85.6 mm to (21.2, 33.4)
- moved U$10 85.6 mm to (12.6, 44.1)
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Routing:
- net GND: track 219.7 -> 203.5 mm
- net N$75: track 1.01 -> 8.06 mm
- net AIN1-: track 31.3 -> 27.8 mm
- net AIN1+: track 31.0 -> 28.2 mm
- net AIN0-: track 56.5 -> 54.5 mm
- net AIN0+: track 55.3 -> 53.9 mm
- net CV4: track 33.7 -> 33.0 mm
